File: hardware/KiCAD/PiBot.sch (KiCad schematic (older format))
At the start: 1 part

Commit message: adding power updates
Parts:
- added C?: 0.1uF, symbol C
Connections:
- net +3V3: now reaches U?.1 (VDD)
- net +3V3: now also U?.13 (VDDA), U?.30 (VDD), U?.48 (VDD), C?.1
- net GND: now reaches U?.16 (VSSA)
- net GND: now also U?.31 (VSS), U?.4 (VSS), U?.47 (VSS), C?.2
- no-connect marks 0 -> 2
Changed lines of the file:
@@
 LIBS:valves
 LIBS:mk20dx64vlh7
+LIBS:PiBot-cache
 EELAYER 25 0
 EELAYER END
@@
 	1    0    0    -1
 $EndComp
+$Comp
+L +3.3V #PWR?
+U 1 1 582E9263
+P 2150 650
+F 0 "#PWR?" H 2150 500 50  0001 C CNN
+F 1 "+3.3V" H 2000 700 50  0000 C CNN
+F 2 "" H 2150 650 50  0000 C CNN
+F 3 "" H 2150 650 50  0000 C CNN
+	1    2150 650
+	1    0    0    -1
+$EndComp
+$Comp
+L GND #PWR?
+U 1 1 582E92A4
+P 2100 3000
+F 0 "#PWR?" H 2100 2750 50  0001 C CNN
+F 1 "GND" H 2100 2850 50  0000 C CNN
+F 2 "" H 2100 3000 50  0000 C CNN
+F 3 "" H 2100 3000 50  0000 C CNN
+	1    2100 3000
+	1    0    0    -1
+$EndComp
+Wire Wire Line
+	2050 3000 2400 3000
+Connection ~ 2100 3000
+Wire Wire Line
+	2150 650  2150 1050
+Wire Wire Line
+	2150 1050 1950 1050
+Connection ~ 2100 1050
+Connection ~ 2050 1050
+NoConn ~ 3150 1250
+Connection ~ 2150 3000
+NoConn ~ 2350 1050
+$Comp
+L C C?
+U 1 1 582E9431
+P 1800 800
+F 0 "C?" H 1825 900 50  0000 L CNN
+F 1 "0.1uF" H 1825 700 50  0000 L CNN
+F 2 "" H 1838 650 50  0000 C CNN
+F 3 "" H 1800 800 50  0000 C CNN
+	1    1800 800
+	1    0    0    -1
+$EndComp
+$Comp
+L GND #PWR?
+U 1 1 582E946B
+P 1800 950
+F 0 "#PWR?" H 1800 700 50  0001 C CNN
+F 1 "GND" H 1700 950 50  0000 C CNN
+F 2 "" H 1800 950 50  0000 C CNN
+F 3 "" H 1800 950 50  0000 C CNN
+	1    1800 950
+	1    0    0    -1
+$EndComp
+Wire Wire Line
+	2150 650  1800 650
 $EndSCHEMATC

Commit message: Added Motor Driver and Cleanup
Added motor driver chip to PiBot KiCad library and also clean up repo adding files to gitignore that are not crucial to the project
Parts:
- added U? (x2): MC33926PNB, symbol MC33926PNB
Connections:
- net labels added: +BATT, GNDA
- wire segments 4 -> 17
Changed lines of the file:
@@
 LIBS:valves
 LIBS:mk20dx64vlh7
+LIBS:PiBot
 LIBS:PiBot-cache
 EELAYER 25 0
@@
 	1    0    0    -1
 $EndComp
+$Comp
+L MC33926PNB U?
+U 1 1 58301234
+P 4650 650
+F 0 "U?" H 4800 450 60  0000 C CNN
+F 1 "MC33926PNB" V 4650 -150 60  0000 C CNB
+F 2 "" H 4600 650 60  0001 C CNN
+F 3 "" H 4600 650 60  0001 C CNN
+	1    4650 650
+	1    0    0    -1
+$EndComp
+$Comp
+L MC33926PNB U?
+U 1 1 5830127C
+P 4650 2650
+F 0 "U?" H 4800 2450 60  0000 C CNN
+F 1 "MC33926PNB" V 4650 1850 60  0000 C CNB
+F 2 "" H 4600 2650 60  0001 C CNN
+F 3 "" H 4600 2650 60  0001 C CNN
+	1    4650 2650
+	1    0    0    -1
+$EndComp
+$Comp
+L GND #PWR?
+U 1 1 5830134B
+P 4750 2200
+F 0 "#PWR?" H 4750 1950 50  0001 C CNN
+F 1 "GND" H 4750 2050 50  0000 C CNN
+F 2 "" H 4750 2200 50  0000 C CNN
+F 3 "" H 4750 2200 50  0000 C CNN
+	1    4750 2200
+	1    0    0    -1
+$EndComp
+$Comp
+L GNDA #PWR?
+U 1 1 58301453
+P 4500 2200
+F 0 "#PWR?" H 4500 1950 50  0001 C CNN
+F 1 "GNDA" H 4500 2050 50  0000 C CNN
+F 2 "" H 4500 2200 50  0000 C CNN
+F 3 "" H 4500 2200 50  0000 C CNN
+	1    4500 2200
+	1    0    0    -1
+$EndComp
+$Comp
+L GNDA #PWR?
+U 1 1 583017C9
+P 4500 4200
+F 0 "#PWR?" H 4500 3950 50  0001 C CNN
+F 1 "GNDA" H 4500 4050 50  0000 C CNN
+F 2 "" H 4500 4200 50  0000 C CNN
+F 3 "" H 4500 4200 50  0000 C CNN
+	1    4500 4200
+	1    0    0    -1
+$EndComp
+$Comp
+L GND #PWR?
+U 1 1 583017E9
+P 4750 4200
+F 0 "#PWR?" H 4750 3950 50  0001 C CNN
+F 1 "GND" H 4750 4050 50  0000 C CNN
+F 2 "" H 4750 4200 50  0000 C CNN
+F 3 "" H 4750 4200 50  0000 C CNN
+	1    4750 4200
+	1    0    0    -1
+$EndComp
+$Comp
+L +BATT #PWR?
+U 1 1 58301A5C
+P 4550 2800
+F 0 "#PWR?" H 4550 2650 50  0001 C CNN
+F 1 "+BATT" H 4550 2940 50  0000 C CNN
+F 2 "" H 4550 2800 50  0000 C CNN
+F 3 "" H 4550 2800 50  0000 C CNN
+	1    4550 2800
+	1    0    0    -1
+$EndComp
+$Comp
+L +BATT #PWR?
+U 1 1 58301B18
+P 4550 800
+F 0 "#PWR?" H 4550 650 50  0001 C CNN
+F 1 "+BATT" H 4550 940 50  0000 C CNN
+F 2 "" H 4550 800 50  0000 C CNN
+F 3 "" H 4550 800 50  0000 C CNN
+	1    4550 800
+	1    0    0    -1
+$EndComp
+Wire Wire Line
+	2050 3000 2400 3000
+Connection ~ 2100 3000
+Wire Wire Line
+	2150 650  2150 1050
+Wire Wire Line
+	2150 1050 1950 1050
+Connection ~ 2100 1050
+Connection ~ 2050 1050
+Connection ~ 2150 3000
 Wire Wire Line
 	2150 650  1800 650
+Wire Wire Line
+	4600 2200 4850 2200
+Connection ~ 4800 2200
+Connection ~ 4750 2200
+Connection ~ 4700 2200
+Connection ~ 4650 2200
+Wire Wire Line
+	4500 2200 4450 2200
+Wire Wire Line
+	4600 4200 4850 4200
+Connection ~ 4800 4200
+Connection ~ 4750 4200
+Connection ~ 4700 4200
+Connection ~ 4650 4200
+Wire Wire Line
+	4450 4200 4500 4200
+Wire Wire Line
+	4500 800  4650 800
+Connection ~ 4550 800
+Connection ~ 4600 800
+Wire Wire Line
+	4500 2800 4650 2800
+Connection ~ 4550 2800
+Connection ~ 4600 2800
+Wire Wire Line
+	5000 1200 5000 1350
+Connection ~ 5000 1250
+Connection ~ 5000 1300
+Wire Wire Line
+	5000 1650 5000 1800
+Connection ~ 5000 1700
+Connection ~ 5000 1750
+Wire Wire Line
+	5000 3200 5000 3350
+Connection ~ 5000 3250
+Connection ~ 5000 3300
+Wire Wire Line
+	5000 3650 5000 3800
+Connection ~ 5000 3700
+Connection ~ 5000 3750
 $EndSCHEMATC

Commit message: Added Motor and Encoder shematic
Also added preliminary wiring and change grounds to better illustrate what the grounds were used for
Parts:
- added C? (x2): 0.1uF, symbol C
- added U? (x2): Motor, symbol Motor
Connections:
- net labels added: GNDPWR
- net labels removed: GNDA
- wire segments 17 -> 58

Commit message: adding in PQFN package for motor driver
Parts:
- U? (x2): footprint (none) -> KiCAD_lib:PQFN-32-EP-0.8mm
Connections:
- net labels added: left_encA, left_encB, right_encA, right_encB
- wire segments 58 -> 70
Changed lines of the file:
@@
 LIBS:mk20dx64vlh7
 LIBS:PiBot
+LIBS:PiBot-cache
 EELAYER 25 0
 EELAYER END
@@
 F 0 "U?" H 4800 450 60  0000 C CNN
 F 1 "MC33926PNB" V 4650 -150 60  0000 C CNB
-F 2 "" H 4600 650 60  0001 C CNN
+F 2 "KiCAD_lib:PQFN-32-EP-0.8mm" H 4600 650 60  0001 C CNN
 F 3 "" H 4600 650 60  0001 C CNN
 	1    4650 650
@@
 F 0 "U?" H 4800 2450 60  0000 C CNN
 F 1 "MC33926PNB" V 4650 1850 60  0000 C CNB
-F 2 "" H 4600 2650 60  0001 C CNN
+F 2 "KiCAD_lib:PQFN-32-EP-0.8mm" H 4600 2650 60  0001 C CNN
 F 3 "" H 4600 2650 60  0001 C CNN
 	1    4650 2650
@@
 	1    0    0    -1
 $EndComp
+Wire Wire Line
+	5600 1450 5650 1450
+Wire Wire Line
+	5650 1450 5650 1100
+Wire Wire Line
+	5650 1100 5700 1100
+Wire Wire Line
+	5600 1500 5650 1500
+Wire Wire Line
+	5650 1500 5650 1900
+Wire Wire Line
+	5650 1900 5700 1900
+Text GLabel 5700 1900 2    60   Input ~ 0
+left_encB
+Text GLabel 5700 1100 2    60   Input ~ 0
+left_encA
+Wire Wire Line
+	5550 3450 5600 3450
+Wire Wire Line
+	5600 3450 5600 3100
+Wire Wire Line
+	5600 3100 5650 3100
+Wire Wire Line
+	5550 3500 5600 3500
+Wire Wire Line
+	5600 3500 5600 3900
+Wire Wire Line
+	5600 3900 5650 3900
+Text GLabel 5650 3100 2    60   Input ~ 0
+right_encA
+Text GLabel 5650 3900 2    60   Input ~ 0
+right_encB
 $EndSCHEMATC

Commit message: moving the micro to the PiBot lib
Parts:
- removed U?: MK20DX64VLH7, Housings_QFP:LQFP-64_10x10mm_Pitch0.5mm, symbol MK20DX64VLH7
- added U?: MK20DX64VLH7, symbol MK20DX64VLH7
Changed lines of the file:
@@
 LIBS:contrib
 LIBS:valves
-LIBS:mk20dx64vlh7
 LIBS:PiBot
 LIBS:PiBot-cache
@@
 $EndDescr
 $Comp
-L MK20DX64VLH7 U?
-U 1 1 582D41FB
-P 2250 2050
-F 0 "U?" H 2900 3000 60  0000 C CNN
-F 1 "MK20DX64VLH7" H 2300 2250 60  0000 C CNB
-F 2 "Housings_QFP:LQFP-64_10x10mm_Pitch0.5mm" H 2250 2050 60  0001 C CNN
-F 3 "" H 2250 2050 60  0001 C CNN
-	1    2250 2050
-	1    0    0    -1
-$EndComp
-$Comp
 L +3.3V #PWR?
 U 1 1 582E9263
@@
 Text GLabel 5650 3900 2    60   Input ~ 0
 right_encB
+$Comp
+L MK20DX64VLH7 U?
+U 1 1 5833AEE0
+P 2250 2050
+F 0 "U?" H 2900 3000 60  0000 C CNN
+F 1 "MK20DX64VLH7" H 2300 2250 60  0000 C CNB
+F 2 "" H 2250 2050 60  0001 C CNN
+F 3 "" H 2250 2050 60  0001 C CNN
+	1    2250 2050
+	1    0    0    -1
+$EndComp
 $EndSCHEMATC

Commit message: Added Molex Micro SD card schematic symbol
Parts:
- added U?: MolexMicroSD, symbol MolexMicroSD
Connections:
- wire segments 70 -> 43
Changed lines of the file:
@@
 $EndComp
 Wire Wire Line
-	2050 3000 2100 3000
-Wire Wire Line
-	2100 3000 2150 3000
-Wire Wire Line
-	2150 3000 2400 3000
+	2050 3000 2400 3000
 Connection ~ 2100 3000
 Wire Wire Line
 	2150 1050 2150 650
 Wire Wire Line
-	1950 1050 2050 1050
-Wire Wire Line
-	2050 1050 2100 1050
-Wire Wire Line
-	2100 1050 2150 1050
+	1950 1050 2150 1050
 Connection ~ 2100 1050
 Connection ~ 2050 1050
@@
 	2150 650  1800 650
 Wire Wire Line
-	4600 2200 4650 2200
-Wire Wire Line
-	4650 2200 4700 2200
-Wire Wire Line
-	4700 2200 4750 2200
-Wire Wire Line
-	4750 2200 4800 2200
-Wire Wire Line
-	4800 2200 4850 2200
+	4600 2200 4850 2200
 Connection ~ 4800 2200
 Connection ~ 4750 2200
@@
 	4500 2200 4450 2200
 Wire Wire Line
-	4600 4200 4650 4200
-Wire Wire Line
-	4650 4200 4700 4200
-Wire Wire Line
-	4700 4200 4750 4200
-Wire Wire Line
-	4750 4200 4800 4200
-Wire Wire Line
-	4800 4200 4850 4200
+	4600 4200 4850 4200
 Connection ~ 4800 4200
 Connection ~ 4750 4200
@@
 	4450 4200 4500 4200
 Wire Wire Line
-	4500 800  4550 800
-Wire Wire Line
-	4550 800  4600 800
-Wire Wire Line
-	4600 800  4650 800
+	4500 800  4650 800
 Connection ~ 4550 800
 Connection ~ 4600 800
 Wire Wire Line
-	4500 2800 4550 2800
-Wire Wire Line
-	4550 2800 4600 2800
-Wire Wire Line
-	4600 2800 4650 2800
+	4500 2800 4650 2800
 Connection ~ 4550 2800
 Connection ~ 4600 2800
@@
 $EndComp
 Wire Wire Line
-	5000 3550 5000 3650
-Wire Wire Line
-	5000 3650 5000 3700
-Wire Wire Line
-	5000 3700 5000 3750
-Wire Wire Line
-	5000 3750 5000 3800
+	5000 3550 5000 3800
 Connection ~ 5000 3750
 Connection ~ 5000 3700
@@
 	5000 3400 5050 3400
 Wire Wire Line
-	5000 3200 5000 3250
-Wire Wire Line
-	5000 3250 5000 3300
-Wire Wire Line
-	5000 3300 5000 3350
-Wire Wire Line
-	5000 3350 5000 3400
+	5000 3200 5000 3400
 Connection ~ 5000 3350
 Connection ~ 5000 3300
 Connection ~ 5000 3250
 Wire Wire Line
-	5000 1200 5000 1250
-Wire Wire Line
-	5000 1250 5000 1300
-Wire Wire Line
-	5000 1300 5000 1350
-Wire Wire Line
-	5000 1350 5000 1400
+	5000 1200 5000 1400
 Wire Wire Line
 	5000 1400 5100 1400
@@
 	5100 1550 5000 1550
 Wire Wire Line
-	5000 1550 5000 1650
-Wire Wire Line
-	5000 1650 5000 1700
-Wire Wire Line
-	5000 1700 5000 1750
-Wire Wire Line
-	5000 1750 5000 1800
+	5000 1550 5000 1800
 $Comp
 L C C?
@@
 	1    0    0    -1
 $EndComp
+$Comp
+L MolexMicroSD U?
+U 1 1 5834082C
+P 5050 5750
+F 0 "U?" H 5450 6000 60  0000 C CNN
+F 1 "MolexMicroSD" H 5050 5750 60  0000 C CNB
+F 2 "" H 4700 6100 60  0001 C CNN
+F 3 "" H 4700 6100 60  0001 C CNN
+	1    5050 5750
+	1    0    0    -1
+$EndComp
+$Comp
+L GND #PWR?
+U 1 1 58340D24
+P 5050 6050
+F 0 "#PWR?" H 5050 5800 50  0001 C CNN
+F 1 "GND" H 5050 5900 50  0000 C CNN
+F 2 "" H 5050 6050 50  0000 C CNN
+F 3 "" H 5050 6050 50  0000 C CNN
+	1    5050 6050
+	1    0    0    -1
+$EndComp
+Wire Wire Line
+	5000 6050 5050 6050
+$Comp
+L +3.3V #PWR?
+U 1 1 5834102E
+P 5050 5450
+F 0 "#PWR?" H 5050 5300 50  0001 C CNN
+F 1 "+3.3V" H 4900 5500 50  0000 C CNN
+F 2 "" H 5050 5450 50  0000 C CNN
+F 3 "" H 5050 5450 50  0000 C CNN
+	1    5050 5450
+	1    0    0    -1
+$EndComp
