File: hardware/KiCAD/PiBot.sch (KiCad schematic (older format))
At the start: 71 parts

Commit message: Add micro and JTAG
Added micro schematic symbol and wired up to power and JTAG using the defined 10-pin ARM jtag standard
Parts:
- added C?: 0.01uF, symbol C
- added C?: 0.1uF, symbol C
- added C?: 1uF, symbol C
- added P?: CONN_02X05, symbol CONN_02X05
- added U?: MKL03ZxxVFK4, symbol MKL03ZxxVFK4
- added U?: MC33926PNB, PiBot:PQFN-32-EP-0.8mm, symbol MC33926PNB
Connections:
- net labels added: RESET, SWCLK, SWDIO, SWO
- wire segments 255 -> 210

Commit message: hooked up KL03 micro and refactored power to a new sheet
Parts:
- removed BT?: Battery, symbol Battery
- removed C? (x3): 0.1uF, symbol C
- removed C? (x2): 10uF, symbol C
- removed C?: 10pf, symbol C
- removed C? (x3): 22uf, symbol C
- removed D? (x2): DZ2J051M0L, symbol ZENERsmall
- removed D?: DZ2J075M0L, symbol ZENERsmall
- removed L?: 1 uH, symbol INDUCTOR_SMALL
- removed R? (x2): 1M, symbol R_Small
- removed R?: 111k, symbol R_Small
- removed R?: 0R, symbol R
- removed R?: NP, symbol R_Small
- removed R? (x3): 0, symbol R_Small
- removed SW?: SPST, symbol SPST
- removed U?: DMG2302U, symbol DMG2302U
- removed U?: TPS63060, symbol TPS63060
- removed W?: TP, symbol TEST_1P
- added C? (x2): 0.1uF, symbol C
- C?: value 0.01uF -> 10nF
Connections:
- net labels removed: +BATT_ISOLATED, BATT_GND_TERM, BATT_V+_TERM, PSU_FB, PSU_IND, PSU_VOUT
- wire segments 210 -> 174
Other:
- note added: "PTA5 - TPM0_CH1 SPI0_SS_b\nPTA6 - TPM0_CH0 SPI0_MISO\nPTB10 - TPM0_CH1 SPI0_SS_b\nPTB11 - TPM0_CH0 SPI0_MISO\nPTB5 - TPM1_CH1 CMP0_IN1\nPTA12 - TPM1_CH0 TPM_CLKIN0\n"
- note added: "PWM Pins\n"
- moved on the sheet: C?

Commit message: update schematic symbols that were out of date
Parts:
- D?: symbol ZENER -> D_Zener
- PTC?: symbol F_Small -> Polyfuse_Small
Connections:
- wire segments 174 -> 185
Changed lines of the file:
@@
 LIBS:PiBot
 LIBS:PiBot-cache
-EELAYER 26 0
+EELAYER 25 0
 EELAYER END
 $Descr A4 11693 8268
@@
 $EndComp
 $Comp
-L F_Small PTC?
+L Polyfuse_Small PTC?
 U 1 1 58579C3D
 P 1800 1400
@@
 F 5 "http://www.digikey.com/product-detail/en/bel-fuse-inc/0ZCJ0050FF2G/507-1802-1-ND/4156236" H 1800 1400 60  0001 C CNN "DigiKey Link"
 	1    1800 1400
-	-1   0    0    -1
-$EndComp
-$Comp
-L ZENER D?
+	0    1    -1   0
+$EndComp
+$Comp
+L D_Zener D?
 U 1 1 58579C3E
 P 1300 1600
@@
 Wire Wire Line
 	7750 3900 7700 3900
+Wire Wire Line
+	600  5600 600  5650
+Wire Wire Line
+	600  5650 800  5650
+Wire Wire Line
+	600  5300 600  5250
+Wire Wire Line
+	600  5250 800  5250
+Wire Wire Line
+	800  4550 650  4550
+Wire Wire Line
+	650  4550 650  4500
+Wire Wire Line
+	650  4200 650  4150
+Wire Wire Line
+	650  4150 800  4150
+Wire Wire Line
+	10650 4700 10600 4700
+Wire Wire Line
+	1300 1750 1300 1800
+Wire Wire Line
+	1300 1450 1300 1400
 $EndSCHEMATC

Commit message: remove old mag and add accel, mag, gyro
Parts:
- removed C?: 0.1uF, symbol C
- removed U?: LIS3MDL, symbol LIS3MDL
- added C?: 10nF, symbol C
- added C? (x2): 0.1uF, symbol C
- added C? (x2): 1uF, symbol C
- added C? (x3): 10uF, symbol C
- added C?: 4.7uF, symbol C
- added C?: 0.22uF, symbol C
- added NP, NP?, R? (x2): 0R, symbol R
- added U?: L3GD20H, symbol L3GD20H
- added U?: LSM303DTR, symbol LSM303DTR
Connections:
- wire segments 185 -> 218

Commit message: Add bumpers, user LED, and hall sensors
Parts:
- removed NP, NP?, R? (x2): 0R, symbol R
- added C? (x6): 0.1uF, symbol C
- added JP? (x7): Jumper_NC_Small, symbol Jumper_NC_Small
- added JP? (x7): Jumper_NO_Small, symbol Jumper_NO_Small
- added R? (x8): 10k, symbol R
- added SW? (x2): SW_SPDT, symbol SW_SPDT
- added U? (x4): AH3772, symbol AH3772
Connections:
- net labels added: front_bumper, rear_bumper, user_LED
- net labels removed: USER_LED_0
- wire segments 218 -> 357
- no-connect marks 6 -> 12
Other:
- note added: "Bumpers"
- note added: "Power"
- moved on the sheet: C?
