File: hardware/KiCAD/PiBot.sch (KiCad schematic (older format))
At the start: 97 parts

Commit message: Organize schematic into multiple sheets
Parts:
- removed C? (x14): 0.1uF, symbol C
- removed C?: 10nF, symbol C
- removed C? (x2): 1uF, symbol C
- removed C? (x2): 10uF, symbol C
- removed C?: 4.7uF, symbol C
- removed C?: 0.22uF, symbol C
- removed JP? (x6): Jumper_NC_Small, symbol Jumper_NC_Small
- removed JP? (x6): Jumper_NO_Small, symbol Jumper_NO_Small
- removed R? (x13): 10k, symbol R
- removed R? (x2): 0R, symbol R
- removed SW? (x2): SW_SPDT, symbol SW_SPDT
- removed U? (x3): MC33926PNB, PiBot:PQFN-32-EP-0.8mm, symbol MC33926PNB
- removed U? (x2): BH1745NUC, PiBot:WSON008X2120, symbol BH1745NUC
- removed U? (x2): Motor, symbol Motor
- removed U?: L3GD20H, symbol L3GD20H
- removed U?: LSM303DTR, symbol LSM303DTR
- removed U? (x4): AH3772, symbol AH3772
- removed W? (x2): TP, symbol TEST_1P
- D? (x4): symbol LED -> LED-RESCUE-PiBot
- R? (x2): value 330R -> 62R
- R?: value 330R -> 150R
- R?: value 330R -> 200R
Connections:
- net labels removed: COLOR_INT_A, COLOR_INT_B, GNDPWR
- wire segments 357 -> 120
- no-connect marks 12 -> 3
Other:
- note added: "*All LED's PN: XZVG45S-9"
- note added: "Debug + Expansion"
- note added: "Motors"
- note added: "SD Card"
- note added: "Sensors"
- note removed: "Bumpers"
- note removed: "Enable Motor\nDrivers if our\n5v line is up"
- note removed: "FB_L/R are feedback analog lines for\nsensing the amount of current the motor\ndriver is sending. Solder the 0 ohm and\ndesolder the 10k to ground for use."
- moved on the sheet: C?

Commit message: Fix Library dependancies
Connections:
- wire segments 120 -> 103
Changed lines of the file:
@@
 EESchema Schematic File Version 2
 LIBS:PiBot-rescue
-LIBS:power
-LIBS:device
-LIBS:transistors
-LIBS:conn
-LIBS:linear
-LIBS:regul
-LIBS:74xx
-LIBS:cmos4000
-LIBS:adc-dac
-LIBS:memory
-LIBS:xilinx
-LIBS:microcontrollers
-LIBS:dsp
-LIBS:microchip
-LIBS:analog_switches
-LIBS:motorola
-LIBS:texas
-LIBS:intel
-LIBS:audio
-LIBS:interface
-LIBS:digital-audio
-LIBS:philips
-LIBS:display
-LIBS:cypress
-LIBS:siliconi
-LIBS:opto
-LIBS:atmel
-LIBS:contrib
-LIBS:valves
 LIBS:PiBot
-LIBS:74xgxx
-LIBS:ac-dc
-LIBS:actel
-LIBS:allegro
-LIBS:Altera
-LIBS:analog_devices
-LIBS:battery_management
-LIBS:bbd
-LIBS:bosch
-LIBS:brooktre
-LIBS:cmos_ieee
-LIBS:dc-dc
-LIBS:diode
-LIBS:elec-unifil
-LIBS:ESD_Protection
-LIBS:ftdi
-LIBS:gennum
-LIBS:graphic
-LIBS:hc11
-LIBS:ir
-LIBS:Lattice
-LIBS:logo
-LIBS:maxim
-LIBS:mechanical
-LIBS:microchip_dspic33dsc
-LIBS:microchip_pic10mcu
-LIBS:microchip_pic12mcu
-LIBS:microchip_pic16mcu
-LIBS:microchip_pic18mcu
-LIBS:microchip_pic32mcu
-LIBS:motor_drivers
-LIBS:motors
-LIBS:msp430
-LIBS:nordicsemi
-LIBS:nxp_armmcu
-LIBS:onsemi
-LIBS:Oscillators
-LIBS:powerint
-LIBS:Power_Management
-LIBS:pspice
-LIBS:references
-LIBS:relays
-LIBS:rfcom
-LIBS:sensors
-LIBS:silabs
-LIBS:stm8
-LIBS:stm32
-LIBS:supertex
-LIBS:switches
-LIBS:transf
-LIBS:ttl_ieee
-LIBS:video
-LIBS:wiznet
-LIBS:Worldsemi
-LIBS:Xicor
-LIBS:zetex
-LIBS:Zilog
 LIBS:PiBot-cache
 EELAYER 25 0
@@
 	4400 2050 4400 2100
 Wire Wire Line
-	1850 2850 1900 2850
-Wire Wire Line
-	1900 2850 1950 2850
+	1850 2850 1950 2850
 Wire Wire Line
 	1850 2900 1850 2850
@@
 	2100 3250 2100 2750
 Wire Wire Line
-	1800 3250 1950 3250
-Wire Wire Line
-	1950 3250 2100 3250
+	1800 3250 2100 3250
 Connection ~ 1850 3350
 Wire Wire Line
@@
 	2150 3350 2150 2850
 Wire Wire Line
-	1800 3350 1850 3350
-Wire Wire Line
-	1850 3350 2150 3350
+	1800 3350 2150 3350
 Wire Wire Line
 	1950 3150 1950 3250
 Wire Wire Line
-	4250 5000 4300 5000
-Wire Wire Line
-	4300 5000 4700 5000
-Wire Wire Line
-	4600 4900 4650 4900
-Wire Wire Line
-	4650 4900 4700 4900
+	4250 5000 4700 5000
+Wire Wire Line
+	4600 4900 4700 4900
 Wire Wire Line
 	4700 4900 4700 4950
 Wire Wire Line
-	5850 4900 5950 4900
-Wire Wire Line
-	5950 4900 6000 4900
-Wire Wire Line
-	5850 5050 6300 5050
-Wire Wire Line
-	6300 5050 6350 5050
-Wire Wire Line
-	1800 1950 1950 1950
-Wire Wire Line
-	1950 1950 2150 1950
+	5850 4900 6000 4900
+Wire Wire Line
+	5850 5050 6350 5050
+Wire Wire Line
+	1800 1950 2150 1950
 Connection ~ 1950 1950
 Wire Wire Line
@@
 	3950 3050 4000 3050
 Wire Wire Line
-	4300 3050 4350 3050
-Wire Wire Line
-	4350 3050 4400 3050
+	4300 3050 4400 3050
 Connection ~ 4350 3050
 Wire Wire Line
@@
 	2050 1850 2150 1850
 Wire Wire Line
-	8400 1250 8550 1250
-Wire Wire Line
-	8550 1250 8850 1250
-Wire Wire Line
-	8850 1250 9100 1250
-Wire Wire Line
-	9100 1250 9350 1250
+	8400 1250 9350 1250
 Wire Wire Line
 	8400 1250 8400 1550
 Wire Wire Line
-	8550 1550 8850 1550
-Wire Wire Line
-	8850 1550 9100 1550
-Wire Wire Line
-	9100 1550 9350 1550
+	8550 1550 9350 1550
 Wire Wire Line
 	8850 1550 8850 1600
@@
 	2550 5650 2650 5650
 Wire Wire Line
-	2550 5350 2550 5450
-Wire Wire Line
-	2550 5450 2550 5650
-Wire Wire Line
-	2550 5650 2550 5750
+	2550 5350 2550 5750
 Wire Wire Line
 	2650 5450 2550 5450
@@
 $EndComp
 Wire Wire Line
-	6450 2800 6450 2850
-Wire Wire Line
-	6450 2850 6450 2900
+	6450 2800 6450 2900
 Wire Wire Line
 	6450 2850 7000 2850

Commit message: Remove user LED and add battery monitor
user LED was sacraficed to make room for battery voltage monitor circuit
Parts:
- removed D?: LED, symbol LED-RESCUE-PiBot
- removed R?: 62R, symbol R
- added C?: 10uF, symbol C
- added D?: 3.3V, symbol D_Zener_Small
- added R?: 10k, symbol R
- added R?: 15k, symbol R
Connections:
- net labels removed: user_LED
- wire segments 103 -> 127
Other:
- note added: "2.5:1 voltage divider"
- note removed: "LED 1\n"

Commit message: Fix errors in schematic
- Fix motor feedback circuit
- Replace micro SD card with standard symbol
- Replace some 0ohm's with cuttable traces
- Clean up motor sheet
Parts:
- removed U?: MolexMicroSD, symbol MolexMicroSD
- removed W? (x3): TP, symbol TEST_1P
- removed W?: TEST_1P, symbol TEST_1P
- added C?: 100uF, symbol C
- added C?: 10uF, symbol C
- added C?: 1uF, symbol C
- added CON?: Micro_SD_Card, symbol Micro_SD_Card
Connections:
- wire segments 127 -> 133

Commit message: Minor cleanup
Other:
- note added: "On Feather boards, VBUS connects \ndirectly to USB power. This is protection \ncircuitry so we don't blow our computers \n(or the feather circuitry)."
- note removed: "On Feather boards, VBUS connects directly to USB\npower. This is protection circuitry so we don't blow\nour computers (or the feather circuitry)."
Changed lines of the file:
@@
 Text GLabel 3950 2750 2    39   BiDi ~ 0
 SCK
-Text Notes 1550 800  0    39   ~ 0
-On Feather boards, VBUS connects directly to USB\npower. This is protection circuitry so we don't blow\nour computers (or the feather circuitry).
+Text Notes 500  2350 0    39   ~ 0
+On Feather boards, VBUS connects \ndirectly to USB power. This is protection \ncircuitry so we don't blow our computers \n(or the feather circuitry).
 $Comp
 L GND #PWR?

Commit message: Fix some errors and add test point
Fixed errors with motor pinout and add test points
Parts:
- added D?: LED, symbol LED-RESCUE-PiBot
- added R?: 62R, symbol R
- added TP? (x50): TEST, symbol TEST
- added U?: DMG2302U, symbol DMG2302U
Connections:
- net labels added: MotorR_Inv
- wire segments 133 -> 125
Other:
- note added: "Motors\n OK"
- note added: "Test Points"
- moved on the sheet: C?

Commit message: Minor cleanup; added breakouts for some things
Parts:
- added P?: BREAKOUT, symbol CONN_01X06
- added P?: BREAKOUT, symbol CONN_01X07
- added P?: BREAKOUT, symbol CONN_01X01
Connections:
- net labels added: I2C_LSB_BIT, VBATT_MONITOR
- net labels removed: VREF
- wire segments 125 -> 138
- no-connect marks 3 -> 6
Other:
- note added: "On Feather boards, VBUS\nconnects directly to USB\npower. This is protection \ncircuitry so we don’t blow\nour computers (or the\nfeather circuitry)."
- note removed: "On Feather boards, VBUS connects \ndirectly to USB power. This is protection \ncircuitry so we don't blow our computers \n(or the feather circuitry)."
Changed lines of the file:
@@
 EESchema Schematic File Version 2
-LIBS:PiBot-rescue
 LIBS:power
 LIBS:device
@@
 LIBS:Zilog
 LIBS:PiBot-cache
-EELAYER 25 0
+EELAYER 26 0
 EELAYER END
 $Descr A4 11693 8268
@@
 	1    0    0    -1
 $EndComp
-Text GLabel 4600 1800 2    39   BiDi ~ 0
-VREF
 Text Notes 7350 7500 0    60   ~ 12
 PycoBot (Teensy uPython Robot)
@@
 L +5V #PWR040
 U 1 1 58579C3C
-P 2050 1500
-F 0 "#PWR040" H 2050 1350 50  0001 C CNN
-F 1 "+5V" H 1950 1600 50  0000 C CNN
-F 2 "" H 2050 1500 50  0000 C CNN
-F 3 "" H 2050 1500 50  0000 C CNN
-	1    2050 1500
+P 1750 1500
+F 0 "#PWR040" H 1750 1350 50  0001 C CNN
+F 1 "+5V" H 1650 1600 50  0000 C CNN
+F 2 "" H 1750 1500 50  0000 C CNN
+F 3 "" H 1750 1500 50  0000 C CNN
+	1    1750 1500
 	-1   0    0    -1
 $EndComp
@@
 L Polyfuse_Small PTC?
 U 1 1 58579C3D
-P 2050 1650
-F 0 "PTC?" H 2050 1750 50  0000 C TNN
-F 1 "0.5A" H 2050 1600 50  0000 C TNN
-F 2 "Resistors_SMD:R_1206" H 2050 1650 50  0001 C CNN
-F 3 "" H 2050 1650 50  0000 C CNN
-F 4 "0ZCJ0050FF2G" H 2050 1650 60  0001 C CNN "MPN"
-F 5 "http://www.digikey.com/product-detail/en/bel-fuse-inc/0ZCJ0050FF2G/507-1802-1-ND/4156236" H 2050 1650 60  0001 C CNN "DigiKey Link"
-	1    2050 1650
+P 1750 1650
+F 0 "PTC?" V 1800 1650 50  0000 C TNN
+F 1 "0.5A" V 1650 1700 50  0000 C CNN
+F 2 "Resistors_SMD:R_1206" H 1750 1650 50  0001 C CNN
+F 3 "" H 1750 1650 50  0000 C CNN
+F 4 "0ZCJ0050FF2G" H 1750 1650 60  0001 C CNN "MPN"
+F 5 "http://www.digikey.com/product-detail/en/bel-fuse-inc/0ZCJ0050FF2G/507-1802-1-ND/4156236" H 1750 1650 60  0001 C CNN "DigiKey Link"
+	1    1750 1650
 	-1   0    0    -1
 $EndComp
@@
 L D_Zener D?
 U 1 1 58579C3E
-P 2600 2000
-F 0 "D?" H 2650 1900 50  0000 C CNN
-F 1 "5.1V-1W" H 2650 2100 50  0000 C CNN
-F 2 "Diodes_SMD:SMA_Standard" H 2600 2000 50  0001 C CNN
-F 3 "" H 2600 2000 50  0000 C CNN
-F 4 "SMAZ5V1-13-F" H 2600 2000 60  0001 C CNN "MPN"
-F 5 "http://www.digikey.com/product-detail/en/diodes-incorporated/SMAZ5V1-13-F/SMAZ5V1-FDICT-ND/725074" H 2600 2000 60  0001 C CNN "DigiKey Link"
-	1    2600 2000
+P 2200 2000
+F 0 "D?" H 2350 1950 50  0000 C CNN
+F 1 "5.1V-1W" H 2350 2100 50  0000 C CNN
+F 2 "Diodes_SMD:SMA_Standard" H 2200 2000 50  0001 C CNN
+F 3 "" H 2200 2000 50  0000 C CNN
+F 4 "SMAZ5V1-13-F" H 2200 2000 60  0001 C CNN "MPN"
+F 5 "http://www.digikey.com/product-detail/en/diodes-incorporated/SMAZ5V1-13-F/SMAZ5V1-FDICT-ND/725074" H 2200 2000 60  0001 C CNN "DigiKey Link"
+	1    2200 2000
 	0    -1   1    0
 $EndComp
@@
 L GND #PWR041
 U 1 1 58579C3F
-P 2600 2200
-F 0 "#PWR041" H 2600 1950 50  0001 C CNN
-F 1 "GND" H 2600 2050 50  0001 C CNN
-F 2 "" H 2600 2200 50  0000 C CNN
-F 3 "" H 2600 2200 50  0000 C CNN
-	1    2600 2200
+P 2200 2200
+F 0 "#PWR041" H 2200 1950 50  0001 C CNN
+F 1 "GND" H 2200 2050 50  0001 C CNN
+F 2 "" H 2200 2200 50  0000 C CNN
+F 3 "" H 2200 2200 50  0000 C CNN
+	1    2200 2200
 	-1   0    0    -1
 $EndComp
@@
 L R R?
 U 1 1 58579C45
-P 2600 2850
-F 0 "R?" V 2680 2850 50  0000 C CNN
-F 1 "10k" V 2600 2850 50  0000 C CNN
-F 2 "" V 2530 2850 50  0000 C CNN
-F 3 "" H 2600 2850 50  0000 C CNN
-	1    2600 2850
+P 2600 2900
+F 0 "R?" V 2680 2900 50  0000 C CNN
+F 1 "10k" V 2600 2900 50  0000 C CNN
+F 2 "" V 2530 2900 50  0000 C CNN
+F 3 "" H 2600 2900 50  0000 C CNN
+	1    2600 2900
 	1    0    0    -1
 $EndComp
@@
 L +3.3V #PWR044
 U 1 1 58579C46
-P 2550 2650
-F 0 "#PWR044" H 2550 2500 50  0001 C CNN
-F 1 "+3.3V" H 2400 2700 50  0000 C CNN
-F 2 "" H 2550 2650 50  0000 C CNN
-F 3 "" H 2550 2650 50  0000 C CNN
-	1    2550 2650
+P 2550 2700
+F 0 "#PWR044" H 2550 2550 50  0001 C CNN
+F 1 "+3.3V" H 2400 2750 50  0000 C CNN
+F 2 "" H 2550 2700 50  0000 C CNN
+F 3 "" H 2550 2700 50  0000 C CNN
+	1    2550 2700
 	1    0    0    -1
 $EndComp
@@
 L D_Schottky D?
 U 1 1 58579C47
-P 2300 1800
-F 0 "D?" H 2300 1900 50  0000 C CNN
-F 1 "Schottky" H 2300 1700 50  0000 C CNN
-F 2 "Diodes_SMD:SOD-323" H 2300 1800 50  0001 C CNN
-F 3 "" H 2300 1800 50  0000 C CNN
-F 4 "CUS10S30H3FCT-ND" H 2300 1800 60  0001 C CNN "MPN"
-F 5 "230mV @ 100mA" H 2300 1800 60  0001 C CNN "Vf"
-	1    2300 1800
+P 1950 1800
+F 0 "D?" H 1900 1900 50  0000 C CNN
+F 1 "Schottky" H 1950 1700 50  0000 C CNN
+F 2 "Diodes_SMD:SOD-323" H 1950 1800 50  0001 C CNN
+F 3 "" H 1950 1800 50  0000 C CNN
+F 4 "CUS10S30H3FCT-ND" H 1950 1800 60  0001 C CNN "MPN"
+F 5 "230mV @ 100mA" H 1950 1800 60  0001 C CNN "Vf"
+	1    1950 1800
 	-1   0    0    -1
 $EndComp
@@
 Text GLabel 4600 2600 2    39   BiDi ~ 0
 SCK
-Text Notes 1150 2200 0    39   ~ 0
-On Feather boards, VBUS connects \ndirectly to USB power. This is protection \ncircuitry so we don't blow our computers \n(or the feather circuitry).
+Text Notes 850  2150 0    39   ~ 0
+On Feather boards, VBUS\nconnects directly to USB\npower. This is protection \ncircuitry so we don’t blow\nour computers (or the\nfeather circuitry).
 $Comp
 L GND #PWR?
@@
 U 1 1 585FB60E
 P 4800 2900
-F 0 "R?" V 4900 2900 50  0000 C CNN
+F 0 "R?" V 4900 2950 50  0000 C CNN
 F 1 "0R" V 4800 2900 50  0000 C CNN
 F 2 "" V 4730 2900 50  0000 C CNN
@@
 	1    0    0    -1
 $EndComp
-Text Label 2650 1800 0    30   ~ 0
+Text Label 2250 1800 0    30   ~ 0
 F_VBUS
 $Comp
@@
 FB_L
 Wire Wire Line
-	5050 1900 5050 1950
-Wire Wire Line
-	2500 2700 2600 2700
-Wire Wire Line
-	2500 2750 2500 2700
+	2500 2750 2600 2750
 Connection ~ 2600 3100
 Wire Wire Line
@@
 	2450 3200 2800 3200
 Wire Wire Line
-	2600 3000 2600 3100
-Wire Wire Line
-	2450 1800 2800 1800
-Connection ~ 2600 1800
+	2600 3050 2600 3100
+Wire Wire Line
+	2100 1800 2800 1800
+Connection ~ 2200 1800
 Wire Wire Line
 	4600 1600 4650 1600
@@
 	9450 2500 9400 2500
 Wire Wire Line
-	2600 2150 2600 2200
-Wire Wire Line
-	2600 1850 2600 1800
+	2200 2150 2200 2200
+Wire Wire Line
+	2200 1850 2200 1800
 $Comp
 L C C?
@@
 U 1 1 586B1E97
 P 6000 2550
-F 0 "JP?" H 6000 2630 50  0000 C CNN
+F 0 "JP?" H 6000 2500 50  0000 C TNN
 F 1 "Jumper_NC_Small" H 6010 2490 50  0001 C CNN
 F 2 "" H 6000 2550 50  0000 C CNN
@@
 	4850 6750 4600 6750
 Wire Wire Line
-	2150 1800 2050 1800
-Wire Wire Line
-	2050 1800 2050 1750
-Wire Wire Line
-	2050 1500 2050 1550
+	1800 1800 1750 1800
+Wire Wire Line
+	1750 1800 1750 1750
+Wire Wire Line
+	1750 1500 1750 1550
 $Comp
 L +3.3V #PWR?
@@
 $EndComp
 Wire Wire Line
-	2550 2650 2550 2700
-Connection ~ 2550 2700
+	2550 2700 2550 2750
+Connection ~ 2550 2750
 Wire Wire Line
 	9450 2200 9400 2200
@@
 Wire Wire Line
 	8300 4350 8450 4350
-Text GLabel 1500 4900 2    39   Output ~ 0
-MotorR_Inv
-Wire Wire Line
-	1500 4900 1400 4900
 Text GLabel 9450 5600 3    39   Output ~ 0
 MotorR_Inv
@@
 Text Notes 7000 4050 0    60   Italic 12
 Test Points
+$Comp
+L CONN_01X06 P?
+U 1 1 586E0430
+P 4850 2250
+F 0 "P?" V 4950 2400 50  0000 L CNN
+F 1 "BREAKOUT" V 4950 1950 50  0000 L CNN
+F 2 "" H 4850 2250 50  0000 C CNN
+F 3 "" H 4850 2250 50  0000 C CNN
+	1    4850 2250
+	1    0    0    -1
+$EndComp
+$Comp
+L CONN_01X07 P?
+U 1 1 586E08CF
+P 2550 2200
+F 0 "P?" V 2650 2450 50  0000 C CNN
+F 1 "BREAKOUT" V 2650 2100 50  0000 C CNN
+F 2 "" H 2550 2200 50  0000 C CNN
+F 3 "" H 2550 2200 50  0000 C CNN
+	1    2550 2200
+	-1   0    0    1
+$EndComp
+Wire Wire Line
+	2750 1900 2800 1900
+Wire Wire Line
+	2800 2000 2750 2000
+Wire Wire Line
+	2750 2100 2800 2100
+Wire Wire Line
+	2800 2200 2750 2200
+Wire Wire Line
+	2750 2300 2800 2300
+Wire Wire Line
+	2800 2400 2750 2400
+Wire Wire Line
+	2750 2500 2800 2500
+Wire Wire Line
+	4600 2500 4650 2500
+Wire Wire Line
+	4650 2400 4600 2400
+Wire Wire Line
+	4600 2300 4650 2300
+Wire Wire Line
+	4650 2200 4600 2200
+Wire Wire Line
+	4600 2100 4650 2100
+Wire Wire Line
+	4650 2000 4600 2000
+NoConn ~ 2650 5550
+NoConn ~ 3150 5550
+$Comp
+L CONN_01X01 P?
+U 1 1 586EA9A5
+P 4750 3300
+F 0 "P?" V 4800 3050 50  0000 L CNN
+F 1 "BREAKOUT" V 4900 3050 50  0000 L CNN
+F 2 "" H 4750 3300 50  0000 C CNN
+F 3 "" H 4750 3300 50  0000 C CNN
+	1    4750 3300
+	0    1    1    0
+$EndComp
+Wire Wire Line
+	4750 3100 4750 3000
+Wire Wire Line
+	4750 3000 4600 3000
+Wire Wire Line
+	5050 1900 5050 1950
+NoConn ~ 4600 1800
+Text Label 6050 2700 0    30   ~ 0
+I2C_LSB_BIT
+Text Label 9550 2600 0    30   ~ 0
+VBATT_MONITOR
 $EndSCHEMATC

Commit message: Split battery into 4 individual batteries
Parts:
- U?: symbol DMG2302U -> DMG2302U-RESCUE-PiBot
Connections:
- wire segments 138 -> 139
- no-connect marks 6 -> 7
Changed lines of the file:
@@
 LIBS:Zilog
 LIBS:PiBot-cache
-EELAYER 26 0
+EELAYER 25 0
 EELAYER END
 $Descr A4 11693 8268
@@
 	2800 6250 2800 6350
 $Comp
-L DMG2302U U?
+L DMG2302U-RESCUE-PiBot U?
 U 1 1 586CD096
 P 2800 7300
@@
 Text Label 9550 2600 0    30   ~ 0
 VBATT_MONITOR
+Wire Wire Line
+	1400 4900 1500 4900
+NoConn ~ 1500 4900
 $EndSCHEMATC
