File: hardware/KiCAD/power.sch (KiCad schematic (older format))
At the start: 25 parts

Commit message: update schematic symbols that were out of date
Parts:
- D? (x3): symbol ZENERsmall -> D_Zener_Small
- L?: symbol INDUCTOR_SMALL -> L
Connections:
- wire segments 90 -> 60
Changed lines of the file:
@@
 LIBS:PiBot
 LIBS:PiBot-cache
-EELAYER 26 0
+EELAYER 25 0
 EELAYER END
 $Descr A4 11693 8268
@@
 $EndComp
 $Comp
-L ZENERsmall D?
+L D_Zener_Small D?
 U 1 1 586935B5
 P 2000 3600
@@
 $EndComp
 $Comp
-L ZENERsmall D?
+L D_Zener_Small D?
 U 1 1 586935B6
 P 2000 3800
@@
 $EndComp
 $Comp
-L INDUCTOR_SMALL L?
+L L L?
 U 1 1 586935B7
 P 5550 2550
 F 0 "L?" H 5400 2650 50  0000 C CNN
-F 1 "1 uH" H 5700 2650 50  0000 C CNN
+F 1 "1 uH" V 5650 2550 50  0000 C CNN
 F 2 "" H 5550 2550 50  0000 C CNN
 F 3 "" H 5550 2550 50  0000 C CNN
 	1    5550 2550
-	1    0    0    -1
+	0    -1   -1   0
 $EndComp
 $Comp
@@
 $EndComp
 $Comp
-L ZENERsmall D?
+L D_Zener_Small D?
 U 1 1 586935C9
 P 3500 3700
@@
 	4800 2350 7000 2350
 Wire Wire Line
-	3100 2900 3100 3200
-Wire Wire Line
-	3100 3200 3100 3250
+	3100 2900 3100 3250
 Wire Wire Line
 	3500 4200 3150 4200
@@
 Connection ~ 3500 3900
 Wire Wire Line
-	3500 3800 3500 3900
-Wire Wire Line
-	3500 3900 3500 4200
+	3500 3800 3500 4200
 Wire Wire Line
 	3800 3500 3800 3550
@@
 Connection ~ 2550 3500
 Wire Wire Line
-	4400 2650 4600 2650
-Wire Wire Line
-	4600 2650 4800 2650
+	4400 2650 4800 2650
 Wire Wire Line
 	4800 3200 4950 3200
@@
 	4700 3100 4950 3100
 Wire Wire Line
-	4700 3100 4700 3300
-Wire Wire Line
-	4700 3300 4700 3350
-Wire Wire Line
-	4150 3300 4400 3300
-Wire Wire Line
-	4400 3300 4700 3300
-Wire Wire Line
-	4700 3300 4950 3300
+	4700 3100 4700 3350
+Wire Wire Line
+	4150 3300 4950 3300
 Connection ~ 6800 2900
 Wire Wire Line
@@
 	6800 3500 6800 3400
 Wire Wire Line
-	6150 2900 6800 2900
-Wire Wire Line
-	6800 2900 7000 2900
-Wire Wire Line
-	7000 2900 7250 2900
-Wire Wire Line
-	7250 2900 7500 2900
-Wire Wire Line
-	7500 2900 7750 2900
-Wire Wire Line
-	7000 2250 7000 2350
-Wire Wire Line
-	7000 2350 7000 2900
-Wire Wire Line
-	6250 3500 6450 3500
-Wire Wire Line
-	6450 3500 6600 3500
-Wire Wire Line
-	6600 3500 6800 3500
-Wire Wire Line
-	6800 3500 7250 3500
-Wire Wire Line
-	7250 3500 7500 3500
-Wire Wire Line
-	7500 3500 7750 3500
+	6150 2900 7750 2900
+Wire Wire Line
+	7000 2250 7000 2900
+Wire Wire Line
+	6250 3500 7750 3500
 Wire Wire Line
 	6450 3100 6450 3500
@@
 Connection ~ 4400 2900
 Wire Wire Line
-	3100 2900 4150 2900
-Wire Wire Line
-	4150 2900 4400 2900
-Wire Wire Line
-	4400 2900 4900 2900
-Wire Wire Line
-	4900 2900 4950 2900
+	3100 2900 4950 2900
 Wire Wire Line
 	6150 2550 6150 2800
 Wire Wire Line
-	5800 2550 6150 2550
+	5700 2550 6150 2550
 Wire Wire Line
 	4950 2550 4950 2800
 Wire Wire Line
-	5300 2550 4950 2550
+	4950 2550 5400 2550
 Wire Wire Line
 	2000 3700 2000 3700
 Connection ~ 3800 3900
 Wire Wire Line
-	3400 3900 3500 3900
-Wire Wire Line
-	3500 3900 3800 3900
-Wire Wire Line
-	3800 3900 4000 3900
-Wire Wire Line
-	3800 3850 3800 3900
-Wire Wire Line
-	3800 3900 3800 3950
+	3400 3900 4000 3900
+Wire Wire Line
+	3800 3850 3800 3950
 Wire Wire Line
 	2550 3500 2550 3550
 Connection ~ 2550 3900
 Wire Wire Line
-	2550 3850 2550 3900
-Wire Wire Line
-	2550 3900 2550 4200
-Wire Wire Line
-	800  3900 2000 3900
-Wire Wire Line
-	2000 3900 2550 3900
-Wire Wire Line
-	2550 3900 2700 3900
+	2550 3850 2550 4200
+Wire Wire Line
+	800  3900 2700 3900
 Connection ~ 3100 3500
 Wire Wire Line
-	3100 3450 3100 3500
-Wire Wire Line
-	3100 3500 3100 3550
-Wire Wire Line
-	1950 3500 2000 3500
-Wire Wire Line
-	2000 3500 2550 3500
-Wire Wire Line
-	2550 3500 3100 3500
-Wire Wire Line
-	3100 3500 3500 3500
-Wire Wire Line
-	3500 3500 3800 3500
+	3100 3450 3100 3550
+Wire Wire Line
+	1950 3500 3800 3500
 Wire Wire Line
 	4150 3300 4150 3200

Commit message: Organize schematic into multiple sheets
Parts:
- BT?: symbol Battery -> Battery-RESCUE-PiBot
Changed lines of the file:
@@
 EESchema Schematic File Version 2
+LIBS:PiBot-rescue
 LIBS:power
 LIBS:device
@@
 $Descr A4 11693 8268
 encoding utf-8
-Sheet 2 2
+Sheet 2 4
 Title ""
 Date ""
@@
 $EndComp
 $Comp
-L Battery BT?
+L Battery-RESCUE-PiBot BT?
 U 1 1 586935B2
 P 800 3700
+AR Path="/586935B2" Ref="BT?"  Part="1"
+AR Path="/5869317C/586935B2" Ref="BT?"  Part="1"
 F 0 "BT?" H 900 3750 50  0000 L CNN
 F 1 "Battery" H 800 3600 50  0000 L CNN

Commit message: add missing documentation
Other:
- moved on the sheet: C?

Commit message: Fix errors in schematic
- Fix motor feedback circuit
- Replace micro SD card with standard symbol
- Replace some 0ohm's with cuttable traces
- Clean up motor sheet
Parts:
- removed R?: NP, symbol R_Small
- added JP?: Jumper_NO_Small, symbol Jumper_NO_Small
Changed lines of the file:
@@
 EESchema Schematic File Version 2
 LIBS:PiBot-rescue
+LIBS:power
+LIBS:device
+LIBS:transistors
+LIBS:conn
+LIBS:linear
+LIBS:regul
+LIBS:74xx
+LIBS:cmos4000
+LIBS:adc-dac
+LIBS:memory
+LIBS:xilinx
+LIBS:microcontrollers
+LIBS:dsp
+LIBS:microchip
+LIBS:analog_switches
+LIBS:motorola
+LIBS:texas
+LIBS:intel
+LIBS:audio
+LIBS:interface
+LIBS:digital-audio
+LIBS:philips
+LIBS:display
+LIBS:cypress
+LIBS:siliconi
+LIBS:opto
+LIBS:atmel
+LIBS:contrib
+LIBS:valves
 LIBS:PiBot
+LIBS:74xgxx
+LIBS:ac-dc
+LIBS:actel
+LIBS:allegro
+LIBS:Altera
+LIBS:analog_devices
+LIBS:battery_management
+LIBS:bbd
+LIBS:bosch
+LIBS:brooktre
+LIBS:cmos_ieee
+LIBS:dc-dc
+LIBS:diode
+LIBS:elec-unifil
+LIBS:ESD_Protection
+LIBS:ftdi
+LIBS:gennum
+LIBS:graphic
+LIBS:hc11
+LIBS:ir
+LIBS:Lattice
+LIBS:logo
+LIBS:maxim
+LIBS:mechanical
+LIBS:microchip_dspic33dsc
+LIBS:microchip_pic10mcu
+LIBS:microchip_pic12mcu
+LIBS:microchip_pic16mcu
+LIBS:microchip_pic18mcu
+LIBS:microchip_pic32mcu
+LIBS:motor_drivers
+LIBS:motors
+LIBS:msp430
+LIBS:nordicsemi
+LIBS:nxp_armmcu
+LIBS:onsemi
+LIBS:Oscillators
+LIBS:powerint
+LIBS:Power_Management
+LIBS:pspice
+LIBS:references
+LIBS:relays
+LIBS:rfcom
+LIBS:sensors
+LIBS:silabs
+LIBS:stm8
+LIBS:stm32
+LIBS:supertex
+LIBS:switches
+LIBS:transf
+LIBS:ttl_ieee
+LIBS:video
+LIBS:wiznet
+LIBS:Worldsemi
+LIBS:Xicor
+LIBS:zetex
+LIBS:Zilog
 LIBS:PiBot-cache
 EELAYER 25 0
@@
 $Comp
 L R_Small R?
-U 1 1 586935CA
-P 4000 5000
-F 0 "R?" V 4100 5050 50  0000 L CNN
-F 1 "NP" V 4100 4900 50  0000 L CNN
-F 2 "" H 4000 5000 50  0000 C CNN
-F 3 "" H 4000 5000 50  0000 C CNN
-	1    4000 5000
-	0    1    1    0
-$EndComp
-$Comp
-L R_Small R?
 U 1 1 586935CB
 P 4050 4150
@@
 Connection ~ 4050 4000
 Connection ~ 5100 3700
+$Comp
+L Jumper_NO_Small JP?
+U 1 1 586DB13F
+P 4000 5000
+F 0 "JP?" H 4000 5080 50  0000 C CNN
+F 1 "Jumper_NO_Small" H 4010 4940 50  0001 C CNN
+F 2 "" H 4000 5000 50  0000 C CNN
+F 3 "" H 4000 5000 50  0000 C CNN
+	1    4000 5000
+	1    0    0    -1
+$EndComp
 $EndSCHEMATC

Commit message: Fix some errors and add test point
Fixed errors with motor pinout and add test points
Parts:
- removed W?: TP, symbol TEST_1P
Changed lines of the file:
@@
 Text Notes 7950 7050 0    60   ~ 12
 MIT License\n
-$Comp
-L TEST_1P W?
-U 1 1 586935CD
-P 5550 3450
-F 0 "W?" H 5450 3700 50  0000 L TNN
-F 1 "TP" H 5400 3600 50  0000 L CNN
-F 2 "" H 5750 3450 50  0000 C CNN
-F 3 "" H 5750 3450 50  0000 C CNN
-	1    5550 3450
-	1    0    0    -1
-$EndComp
 Text Label 7250 3700 0    39   ~ 0
 PSU_VOUT
@@
 	1750 4650 1750 4700
 Connection ~ 3500 4300
-Wire Wire Line
-	5350 3450 5750 3450
 Wire Wire Line
 	5750 4000 5900 4000
@@
 Connection ~ 4750 4700
 Wire Wire Line
-	4350 4700 4950 4700
+	4250 4700 4950 4700
 Wire Wire Line
 	4750 4650 4750 4750
@@
 	3500 4650 3500 5000
 Wire Wire Line
-	1750 4700 3650 4700
+	1750 4700 3750 4700
 Connection ~ 4050 4300
 Wire Wire Line
-	4050 4250 4050 4350
+	4050 4250 4050 4450
 Wire Wire Line
 	2900 4300 4750 4300
@@
 	5850 3800 5850 3700
 Connection ~ 5850 3700
-Connection ~ 5550 3450
 Wire Wire Line
 	5150 3450 5000 3450
@@
 	1    0    0    -1
 $EndComp
+Wire Wire Line
+	5350 3450 5750 3450
 $EndSCHEMATC
