File: hardware/KiCAD/power.sch (KiCad schematic (older format))
At the start: 24 parts

Commit message: Split battery into 4 individual batteries
Parts:
- added BT? (x3): Battery, symbol Battery-RESCUE-PiBot
- U?: symbol DMG2302U -> DMG2302U-RESCUE-PiBot
Connections:
- wire segments 60 -> 94
Changed lines of the file:
@@
 LIBS:Zilog
 LIBS:PiBot-cache
-EELAYER 26 0
+EELAYER 25 0
 EELAYER END
 $Descr A4 11693 8268
@@
 $EndDescr
 $Comp
-L DMG2302U U?
+L DMG2302U-RESCUE-PiBot U?
 U 1 1 586935AF
 P 4000 4700
+AR Path="/586935AF" Ref="U?"  Part="1"
+AR Path="/5869317C/586935AF" Ref="U?"  Part="1"
 F 0 "U?" V 3850 4550 60  0000 C CNN
 F 1 "DMG2302U" V 4190 4700 60  0000 C CNN
@@
 L Battery-RESCUE-PiBot BT?
 U 1 1 586935B2
-P 1750 4500
+P 1350 5000
 AR Path="/586935B2" Ref="BT?"  Part="1"
 AR Path="/5869317C/586935B2" Ref="BT?"  Part="1"
-F 0 "BT?" H 1850 4550 50  0000 L CNN
-F 1 "Battery" H 1750 4400 50  0000 L CNN
-F 2 "" V 1750 4540 50  0000 C CNN
-F 3 "" V 1750 4540 50  0000 C CNN
-	1    1750 4500
+F 0 "BT?" H 1450 5050 50  0000 L CNN
+F 1 "Battery" H 1250 4750 50  0001 L CNN
+F 2 "" V 1350 5040 50  0000 C CNN
+F 3 "" V 1350 5040 50  0000 C CNN
+	1    1350 5000
 	1    0    0    -1
 $EndComp
@@
 Text Label 2100 4700 0    30   ~ 0
 BATT_GND_TERM
-Text Label 1900 4300 2    30   ~ 0
+Text Label 1750 4200 1    30   ~ 0
 BATT_V+_TERM
 Text Label 3550 4300 0    30   ~ 0
@@
 	5750 3150 7950 3150
 Wire Wire Line
-	4050 3700 4050 4050
+	4050 3700 4050 4000
+Wire Wire Line
+	4050 4000 4050 4050
 Wire Wire Line
 	4450 5000 4100 5000
@@
 Connection ~ 4450 4700
 Wire Wire Line
-	4450 4600 4450 5000
+	4450 4600 4450 4700
+Wire Wire Line
+	4450 4700 4450 5000
 Wire Wire Line
 	4750 4300 4750 4350
@@
 	4950 4700 4950 4750
 Connection ~ 2950 4300
-Wire Wire Line
-	1750 4300 1900 4300
-Wire Wire Line
-	1750 4350 1750 4300
 Connection ~ 2950 4700
-Wire Wire Line
-	1750 4650 1750 4700
 Connection ~ 3500 4300
 Wire Wire Line
@@
 	5650 3900 5900 3900
 Wire Wire Line
-	5650 3900 5650 4150
-Wire Wire Line
-	5100 4100 5900 4100
+	5650 3900 5650 4100
+Wire Wire Line
+	5650 4100 5650 4150
+Wire Wire Line
+	5100 4100 5350 4100
+Wire Wire Line
+	5350 4100 5650 4100
+Wire Wire Line
+	5650 4100 5900 4100
 Connection ~ 7750 3700
 Wire Wire Line
@@
 	7750 4300 7750 4200
 Wire Wire Line
-	7100 3700 8700 3700
-Wire Wire Line
-	7950 3050 7950 3700
-Wire Wire Line
-	7200 4300 8700 4300
+	7100 3700 7750 3700
+Wire Wire Line
+	7750 3700 7950 3700
+Wire Wire Line
+	7950 3700 8200 3700
+Wire Wire Line
+	8200 3700 8450 3700
+Wire Wire Line
+	8450 3700 8700 3700
+Wire Wire Line
+	7950 3050 7950 3150
+Wire Wire Line
+	7950 3150 7950 3700
+Wire Wire Line
+	7200 4300 7400 4300
+Wire Wire Line
+	7400 4300 7550 4300
+Wire Wire Line
+	7550 4300 7750 4300
+Wire Wire Line
+	7750 4300 8200 4300
+Wire Wire Line
+	8200 4300 8450 4300
+Wire Wire Line
+	8450 4300 8700 4300
 Wire Wire Line
 	7400 3900 7400 4300
@@
 Connection ~ 5350 3700
 Wire Wire Line
-	4050 3700 5900 3700
+	4050 3700 5100 3700
+Wire Wire Line
+	5100 3700 5350 3700
+Wire Wire Line
+	5350 3700 5850 3700
+Wire Wire Line
+	5850 3700 5900 3700
 Wire Wire Line
 	7100 3350 7100 3600
@@
 Connection ~ 4750 4700
 Wire Wire Line
-	4250 4700 4950 4700
-Wire Wire Line
-	4750 4650 4750 4750
+	4250 4700 4450 4700
+Wire Wire Line
+	4450 4700 4750 4700
+Wire Wire Line
+	4750 4700 4950 4700
+Wire Wire Line
+	4750 4650 4750 4700
+Wire Wire Line
+	4750 4700 4750 4750
 Wire Wire Line
 	3500 4300 3500 4350
 Connection ~ 3500 4700
 Wire Wire Line
-	3500 4650 3500 5000
-Wire Wire Line
-	1750 4700 3750 4700
+	3500 4650 3500 4700
+Wire Wire Line
+	3500 4700 3500 5000
+Wire Wire Line
+	1750 4700 2950 4700
+Wire Wire Line
+	2950 4700 3500 4700
+Wire Wire Line
+	3500 4700 3750 4700
 Connection ~ 4050 4300
 Wire Wire Line
-	4050 4250 4050 4450
-Wire Wire Line
-	2900 4300 4750 4300
+	4050 4250 4050 4300
+Wire Wire Line
+	4050 4300 4050 4450
+Wire Wire Line
+	2900 4300 2950 4300
+Wire Wire Line
+	2950 4300 3500 4300
+Wire Wire Line
+	3500 4300 4050 4300
+Wire Wire Line
+	4050 4300 4450 4300
+Wire Wire Line
+	4450 4300 4750 4300
 Wire Wire Line
 	5100 4100 5100 4000
@@
 Wire Wire Line
 	5350 3450 5750 3450
+$Comp
+L Battery-RESCUE-PiBot BT?
+U 1 1 586E837E
+P 1350 4650
+F 0 "BT?" H 1450 4700 50  0000 L CNN
+F 1 "Battery" H 1200 4900 50  0001 L CNN
+F 2 "" V 1350 4690 50  0000 C CNN
+F 3 "" V 1350 4690 50  0000 C CNN
+	1    1350 4650
+	1    0    0    -1
+$EndComp
+$Comp
+L Battery-RESCUE-PiBot BT?
+U 1 1 586E892D
+P 1350 4300
+F 0 "BT?" H 1450 4350 50  0000 L CNN
+F 1 "Battery" H 1350 4200 50  0001 L CNN
+F 2 "" V 1350 4340 50  0000 C CNN
+F 3 "" V 1350 4340 50  0000 C CNN
+	1    1350 4300
+	1    0    0    -1
+$EndComp
+$Comp
+L Battery-RESCUE-PiBot BT?
+U 1 1 586E8EA5
+P 1350 3950
+F 0 "BT?" H 1450 4000 50  0000 L CNN
+F 1 "Battery" H 1350 3850 50  0001 L CNN
+F 2 "" V 1350 3990 50  0000 C CNN
+F 3 "" V 1350 3990 50  0000 C CNN
+	1    1350 3950
+	1    0    0    -1
+$EndComp
+Wire Wire Line
+	1350 5150 1750 5150
+Wire Wire Line
+	1750 5150 1750 4700
+Wire Wire Line
+	1900 4300 1750 4300
+Wire Wire Line
+	1750 4300 1750 3800
+Wire Wire Line
+	1750 3800 1350 3800
+Wire Wire Line
+	1350 4100 1350 4150
+Wire Wire Line
+	1350 4450 1350 4500
+Wire Wire Line
+	1350 4800 1350 4850
 $EndSCHEMATC

Commit message: Remove all references to rescue library
Parts:
- BT? (x4): symbol Battery-RESCUE-PiBot -> Battery_Cell
- SW?: symbol SPST -> SW_SPST
- U?: symbol DMG2302U-RESCUE-PiBot -> DMG2302U
Connections:
- wire segments 94 -> 65
Changed lines of the file:
@@
 LIBS:zetex
 LIBS:Zilog
-LIBS:PiBot-cache
 EELAYER 25 0
 EELAYER END
@@
 $EndDescr
 $Comp
-L DMG2302U-RESCUE-PiBot U?
+L DMG2302U U?
 U 1 1 586935AF
 P 4000 4700
@@
 $EndComp
 $Comp
-L Battery-RESCUE-PiBot BT?
+L Battery_Cell BT?
 U 1 1 586935B2
-P 1350 5000
+P 1450 5050
 AR Path="/586935B2" Ref="BT?"  Part="1"
 AR Path="/5869317C/586935B2" Ref="BT?"  Part="1"
-F 0 "BT?" H 1450 5050 50  0000 L CNN
-F 1 "Battery" H 1250 4750 50  0001 L CNN
-F 2 "" V 1350 5040 50  0000 C CNN
-F 3 "" V 1350 5040 50  0000 C CNN
-	1    1350 5000
+F 0 "BT?" H 1550 5100 50  0000 L CNN
+F 1 "Battery" H 1350 4800 50  0001 L CNN
+F 2 "" V 1450 5090 50  0000 C CNN
+F 3 "" V 1450 5090 50  0000 C CNN
+	1    1450 5050
 	1    0    0    -1
 $EndComp
@@
 $EndComp
 $Comp
-L SPST SW?
+L SW_SPST SW?
 U 1 1 586935C7
 P 2400 4300
@@
 	5750 3150 7950 3150
 Wire Wire Line
-	4050 3700 4050 4000
-Wire Wire Line
-	4050 4000 4050 4050
+	4050 3700 4050 4050
 Wire Wire Line
 	4450 5000 4100 5000
@@
 Connection ~ 4450 4700
 Wire Wire Line
-	4450 4600 4450 4700
-Wire Wire Line
-	4450 4700 4450 5000
+	4450 4600 4450 5000
 Wire Wire Line
 	4750 4300 4750 4350
@@
 	5650 3900 5900 3900
 Wire Wire Line
-	5650 3900 5650 4100
-Wire Wire Line
-	5650 4100 5650 4150
-Wire Wire Line
-	5100 4100 5350 4100
-Wire Wire Line
-	5350 4100 5650 4100
-Wire Wire Line
-	5650 4100 5900 4100
+	5650 3900 5650 4150
+Wire Wire Line
+	5100 4100 5900 4100
 Connection ~ 7750 3700
 Wire Wire Line
@@
 	7750 4300 7750 4200
 Wire Wire Line
-	7100 3700 7750 3700
-Wire Wire Line
-	7750 3700 7950 3700
-Wire Wire Line
-	7950 3700 8200 3700
-Wire Wire Line
-	8200 3700 8450 3700
-Wire Wire Line
-	8450 3700 8700 3700
-Wire Wire Line
-	7950 3050 7950 3150
-Wire Wire Line
-	7950 3150 7950 3700
-Wire Wire Line
-	7200 4300 7400 4300
-Wire Wire Line
-	7400 4300 7550 4300
-Wire Wire Line
-	7550 4300 7750 4300
-Wire Wire Line
-	7750 4300 8200 4300
-Wire Wire Line
-	8200 4300 8450 4300
-Wire Wire Line
-	8450 4300 8700 4300
+	7100 3700 8700 3700
+Wire Wire Line
+	7950 3050 7950 3700
+Wire Wire Line
+	7200 4300 8700 4300
 Wire Wire Line
 	7400 3900 7400 4300
@@
 Connection ~ 5350 3700
 Wire Wire Line
-	4050 3700 5100 3700
-Wire Wire Line
-	5100 3700 5350 3700
-Wire Wire Line
-	5350 3700 5850 3700
-Wire Wire Line
-	5850 3700 5900 3700
+	4050 3700 5900 3700
 Wire Wire Line
 	7100 3350 7100 3600
@@
 Connection ~ 4750 4700
 Wire Wire Line
-	4250 4700 4450 4700
-Wire Wire Line
-	4450 4700 4750 4700
-Wire Wire Line
-	4750 4700 4950 4700
-Wire Wire Line
-	4750 4650 4750 4700
-Wire Wire Line
-	4750 4700 4750 4750
+	4250 4700 4950 4700
+Wire Wire Line
+	4750 4650 4750 4750
 Wire Wire Line
 	3500 4300 3500 4350
 Connection ~ 3500 4700
 Wire Wire Line
-	3500 4650 3500 4700
-Wire Wire Line
-	3500 4700 3500 5000
-Wire Wire Line
-	1750 4700 2950 4700
-Wire Wire Line
-	2950 4700 3500 4700
-Wire Wire Line
-	3500 4700 3750 4700
+	3500 4650 3500 5000
+Wire Wire Line
+	1750 4700 3750 4700
 Connection ~ 4050 4300
 Wire Wire Line
-	4050 4250 4050 4300
-Wire Wire Line
-	4050 4300 4050 4450
-Wire Wire Line
-	2900 4300 2950 4300
-Wire Wire Line
-	2950 4300 3500 4300
-Wire Wire Line
-	3500 4300 4050 4300
-Wire Wire Line
-	4050 4300 4450 4300
-Wire Wire Line
-	4450 4300 4750 4300
+	4050 4250 4050 4450
+Wire Wire Line
+	2600 4300 4750 4300
 Wire Wire Line
 	5100 4100 5100 4000
@@
 	5350 3450 5750 3450
 $Comp
-L Battery-RESCUE-PiBot BT?
+L Battery_Cell BT?
 U 1 1 586E837E
-P 1350 4650
-F 0 "BT?" H 1450 4700 50  0000 L CNN
-F 1 "Battery" H 1200 4900 50  0001 L CNN
-F 2 "" V 1350 4690 50  0000 C CNN
-F 3 "" V 1350 4690 50  0000 C CNN
-	1    1350 4650
-	1    0    0    -1
-$EndComp
-$Comp
-L Battery-RESCUE-PiBot BT?
+P 1450 4700
+F 0 "BT?" H 1550 4750 50  0000 L CNN
+F 1 "Battery" H 1300 4950 50  0001 L CNN
+F 2 "" V 1450 4740 50  0000 C CNN
+F 3 "" V 1450 4740 50  0000 C CNN
+	1    1450 4700
+	1    0    0    -1
+$EndComp
+$Comp
+L Battery_Cell BT?
 U 1 1 586E892D
-P 1350 4300
-F 0 "BT?" H 1450 4350 50  0000 L CNN
-F 1 "Battery" H 1350 4200 50  0001 L CNN
-F 2 "" V 1350 4340 50  0000 C CNN
-F 3 "" V 1350 4340 50  0000 C CNN
-	1    1350 4300
-	1    0    0    -1
-$EndComp
-$Comp
-L Battery-RESCUE-PiBot BT?
+P 1450 4350
+F 0 "BT?" H 1550 4400 50  0000 L CNN
+F 1 "Battery" H 1450 4250 50  0001 L CNN
+F 2 "" V 1450 4390 50  0000 C CNN
+F 3 "" V 1450 4390 50  0000 C CNN
+	1    1450 4350
+	1    0    0    -1
+$EndComp
+$Comp
+L Battery_Cell BT?
 U 1 1 586E8EA5
-P 1350 3950
-F 0 "BT?" H 1450 4000 50  0000 L CNN
-F 1 "Battery" H 1350 3850 50  0001 L CNN
-F 2 "" V 1350 3990 50  0000 C CNN
-F 3 "" V 1350 3990 50  0000 C CNN
-	1    1350 3950
-	1    0    0    -1
-$EndComp
-Wire Wire Line
-	1350 5150 1750 5150
+P 1450 4000
+F 0 "BT?" H 1550 4050 50  0000 L CNN
+F 1 "Battery" H 1450 3900 50  0001 L CNN
+F 2 "" V 1450 4040 50  0000 C CNN
+F 3 "" V 1450 4040 50  0000 C CNN
+	1    1450 4000
+	1    0    0    -1
+$EndComp
 Wire Wire Line
 	1750 5150 1750 4700
 Wire Wire Line
-	1900 4300 1750 4300
+	1750 4300 2200 4300
 Wire Wire Line
 	1750 4300 1750 3800
 Wire Wire Line
-	1750 3800 1350 3800
-Wire Wire Line
-	1350 4100 1350 4150
-Wire Wire Line
-	1350 4450 1350 4500
-Wire Wire Line
-	1350 4800 1350 4850
+	1750 3800 1450 3800
+Wire Wire Line
+	1750 5150 1450 5150
+Wire Wire Line
+	1450 4800 1450 4850
+Wire Wire Line
+	1450 4500 1450 4450
+Wire Wire Line
+	1450 4150 1450 4100
 $EndSCHEMATC
