File: hardware/KiCAD/power.sch (KiCad schematic (older format))
At the start: 27 parts, among them SW1 SPST, U3 DMG2302U, U4 TPS63060

Commit message: Add battery footprint and assign feather footrprint
Parts:
- BT1, BT2, BT3, BT4: footprint (none) -> PiBot:AA_Batt
Changed lines of the file:
@@
 LIBS:MF_Connectors
 LIBS:PiBot-cache
-EELAYER 26 0
+EELAYER 25 0
 EELAYER END
 $Descr A4 11693 8268
@@
 F 0 "BT4" H 1550 5100 50  0000 L CNN
 F 1 "Battery" H 1350 4800 50  0001 L CNN
-F 2 "" V 1450 5090 50  0001 C CNN
+F 2 "PiBot:AA_Batt" V 1450 5090 50  0001 C CNN
 F 3 "" V 1450 5090 50  0000 C CNN
 	1    1450 5050
@@
 U 1 1 586935BF
 P 5750 3350
-F 0 "R13" V 5650 3300 50  0000 L CNN
-F 1 "1M" V 5750 3350 50  0000 C CNN
+F 0 "R13" H 5780 3370 50  0000 L CNN
+F 1 "1M" V 5750 3300 50  0000 L CNN
 F 2 "Resistors_SMD:R_0402" H 5750 3350 50  0001 C CNN
 F 3 "" H 5750 3350 50  0000 C CNN
@@
 P 7750 3850
 F 0 "R14" H 7780 3870 50  0000 L CNN
-F 1 "1M" V 7750 3850 50  0000 C CNN
+F 1 "1M" V 7750 3800 50  0000 L CNN
 F 2 "Resistors_SMD:R_0402" H 7750 3850 50  0001 C CNN
 F 3 "" H 7750 3850 50  0000 C CNN
@@
 U 1 1 586935C1
 P 7750 4100
-F 0 "R15" V 7950 4000 50  0000 L CNN
-F 1 "111k" V 7850 4100 50  0000 C CNN
+F 0 "R15" H 7780 4120 50  0000 L CNN
+F 1 "111k" V 7750 4000 50  0000 L CNN
 F 2 "Resistors_SMD:R_0402" H 7750 4100 50  0001 C CNN
 F 3 "" H 7750 4100 50  0000 C CNN
@@
 P 7950 2950
 F 0 "R16" V 7850 2900 50  0000 L CNN
-F 1 "0" V 7950 2950 50  0000 C CNN
+F 1 "0" V 7950 2925 50  0000 L CNN
 F 2 "Resistors_SMD:R_0805" H 7950 2950 50  0001 C CNN
 F 3 "" H 7950 2950 50  0000 C CNN
@@
 U 1 1 586DB13F
 P 4000 5000
-F 0 "JP4" H 4000 4900 50  0000 C CNN
+F 0 "JP4" H 4000 5080 50  0000 C CNN
 F 1 "Jumper_NO_Small" H 4010 4940 50  0001 C CNN
 F 2 "" H 4000 5000 50  0001 C CNN
@@
 F 0 "BT3" H 1550 4750 50  0000 L CNN
 F 1 "Battery" H 1300 4950 50  0001 L CNN
-F 2 "" V 1450 4740 50  0001 C CNN
+F 2 "PiBot:AA_Batt" V 1450 4740 50  0001 C CNN
 F 3 "" V 1450 4740 50  0000 C CNN
 	1    1450 4700
@@
 F 0 "BT2" H 1550 4400 50  0000 L CNN
 F 1 "Battery" H 1450 4250 50  0001 L CNN
-F 2 "" V 1450 4390 50  0001 C CNN
+F 2 "PiBot:AA_Batt" V 1450 4390 50  0001 C CNN
 F 3 "" V 1450 4390 50  0000 C CNN
 	1    1450 4350
@@
 F 0 "BT1" H 1550 4050 50  0000 L CNN
 F 1 "Battery" H 1450 3900 50  0001 L CNN
-F 2 "" V 1450 4040 50  0001 C CNN
+F 2 "PiBot:AA_Batt" V 1450 4040 50  0001 C CNN
 F 3 "" V 1450 4040 50  0000 C CNN
 	1    1450 4000

Commit message: Add the rest of the missing footprints, aside from motor
Parts:
- added JP17: Jumper_NC_Small, Oddities:NetTie-I_Connected_SMD, symbol Jumper_NC_Small
- added JP18: Jumper_NO_Small, PiBot:Jumper-NO, symbol Jumper_NO_Small
- added R32: 10k, Resistors_SMD:R_0402, symbol R_Small
- added U17: N-FET, TO_SOT_Packages_SMD:SOT-23, symbol DMG2302U
- BT1, BT2, BT3, BT4: Part Number (none) -> BK-92
- D10: value DZ2J075M0L -> 7.5V; Part Number (none) -> DZ2J075M0L
- D8, D9: value DZ2J051M0L -> 5.1V; footprint Diodes_SMD:SOD-323 -> Diodes_SMD:SMA_Standard; Part Number (none) -> SMAZ5V1-13-F
- JP4: footprint (none) -> PiBot:Jumper-NO
- L1: Part Number (none) -> SRN2512-1R0M
- SW1: footprint (none) -> PiBot:JS202011SCQN; Part Number (none) -> JS202011SCQN
- U3: value DMG2302U -> N-FET; Part Number (none) -> DMG2302U
- U4: footprint Housings_DFN_QFN:DFN-10-1EP_3x3mm_Pitch0.5mm -> PiBot:DFN-10-w_pad
Connections:
- net labels added: -BATT_ISOLATED
- net labels removed: +BATT_ISOLATED
- wire segments 65 -> 74
Other:
- moved on the sheet: C10, C9
