File: hardware/KiCAD/sensors.sch (KiCad schematic (older format))
At the start: 29 parts

Commit message: Fix Library dependancies
Changed lines of the file:
@@
 EESchema Schematic File Version 2
 LIBS:PiBot-rescue
-LIBS:power
-LIBS:device
-LIBS:transistors
-LIBS:conn
-LIBS:linear
-LIBS:regul
-LIBS:74xx
-LIBS:cmos4000
-LIBS:adc-dac
-LIBS:memory
-LIBS:xilinx
-LIBS:microcontrollers
-LIBS:dsp
-LIBS:microchip
-LIBS:analog_switches
-LIBS:motorola
-LIBS:texas
-LIBS:intel
-LIBS:audio
-LIBS:interface
-LIBS:digital-audio
-LIBS:philips
-LIBS:display
-LIBS:cypress
-LIBS:siliconi
-LIBS:opto
-LIBS:atmel
-LIBS:contrib
-LIBS:valves
 LIBS:PiBot
-LIBS:74xgxx
-LIBS:ac-dc
-LIBS:actel
-LIBS:allegro
-LIBS:Altera
-LIBS:analog_devices
-LIBS:battery_management
-LIBS:bbd
-LIBS:bosch
-LIBS:brooktre
-LIBS:cmos_ieee
-LIBS:dc-dc
-LIBS:diode
-LIBS:elec-unifil
-LIBS:ESD_Protection
-LIBS:ftdi
-LIBS:gennum
-LIBS:graphic
-LIBS:hc11
-LIBS:ir
-LIBS:Lattice
-LIBS:logo
-LIBS:maxim
-LIBS:mechanical
-LIBS:microchip_dspic33dsc
-LIBS:microchip_pic10mcu
-LIBS:microchip_pic12mcu
-LIBS:microchip_pic16mcu
-LIBS:microchip_pic18mcu
-LIBS:microchip_pic32mcu
-LIBS:motor_drivers
-LIBS:motors
-LIBS:msp430
-LIBS:nordicsemi
-LIBS:nxp_armmcu
-LIBS:onsemi
-LIBS:Oscillators
-LIBS:powerint
-LIBS:Power_Management
-LIBS:pspice
-LIBS:references
-LIBS:relays
-LIBS:rfcom
-LIBS:sensors
-LIBS:silabs
-LIBS:stm8
-LIBS:stm32
-LIBS:supertex
-LIBS:switches
-LIBS:transf
-LIBS:ttl_ieee
-LIBS:video
-LIBS:wiznet
-LIBS:Worldsemi
-LIBS:Xicor
-LIBS:zetex
-LIBS:Zilog
 LIBS:PiBot-cache
 EELAYER 25 0
@@
 	5800 3200 5500 3200
 Wire Wire Line
-	5500 2800 5500 3200
+	5500 3200 5500 2800
 Wire Wire Line
 	4700 2800 5700 2800

Commit message: add missing documentation
Connections:
- wire segments 75 -> 99
Changed lines of the file:
@@
 Connection ~ 3050 2900
 Wire Wire Line
-	2650 2800 2750 2800
-Wire Wire Line
-	2650 2900 3100 2900
+	2650 2800 2700 2800
+Wire Wire Line
+	2700 2800 2750 2800
+Wire Wire Line
+	2650 2900 3050 2900
+Wire Wire Line
+	3050 2900 3100 2900
 Wire Wire Line
 	1600 1800 1600 1950
@@
 	5500 3200 5500 2800
 Wire Wire Line
-	4700 2800 5700 2800
+	4700 2800 5200 2800
+Wire Wire Line
+	5200 2800 5300 2800
+Wire Wire Line
+	5300 2800 5400 2800
+Wire Wire Line
+	5400 2800 5500 2800
+Wire Wire Line
+	5500 2800 5600 2800
+Wire Wire Line
+	5600 2800 5700 2800
 Connection ~ 5600 2800
 Connection ~ 5500 2800
@@
 Connection ~ 5300 2800
 Wire Wire Line
-	4700 1250 6250 1250
+	4700 1250 5400 1250
+Wire Wire Line
+	5400 1250 5750 1250
+Wire Wire Line
+	5750 1250 6000 1250
+Wire Wire Line
+	6000 1250 6250 1250
 Connection ~ 6000 1250
 Wire Wire Line
-	5400 1200 5400 1550
+	5400 1200 5400 1250
+Wire Wire Line
+	5400 1250 5400 1550
 Connection ~ 5400 1250
 Wire Wire Line
 	5400 1550 5500 1550
 Wire Wire Line
-	5750 1550 6250 1550
+	5750 1550 6000 1550
+Wire Wire Line
+	6000 1550 6250 1550
 Connection ~ 6000 1550
 Wire Wire Line
@@
 	6150 2100 6700 2100
 Wire Wire Line
-	6700 2050 6700 2150
+	6700 2050 6700 2100
+Wire Wire Line
+	6700 2100 6700 2150
 Connection ~ 6700 2100
 Wire Wire Line
@@
 	6700 2350 6700 2400
 Wire Wire Line
-	9300 1550 9800 1550
+	9300 1550 9550 1550
+Wire Wire Line
+	9550 1550 9800 1550
 Connection ~ 9550 1550
 Wire Wire Line
-	8250 1250 9800 1250
+	8250 1250 8950 1250
+Wire Wire Line
+	8950 1250 9300 1250
+Wire Wire Line
+	9300 1250 9550 1250
+Wire Wire Line
+	9550 1250 9800 1250
 Connection ~ 9550 1250
 Wire Wire Line
-	8950 1200 8950 1550
+	8950 1200 8950 1250
+Wire Wire Line
+	8950 1250 8950 1550
 Connection ~ 9300 1250
 Wire Wire Line
@@
 	8350 2100 8250 2100
 Wire Wire Line
-	8750 2800 9150 2800
+	8750 2800 8850 2800
+Wire Wire Line
+	8850 2800 8950 2800
+Wire Wire Line
+	8950 2800 9050 2800
+Wire Wire Line
+	9050 2800 9150 2800
 Connection ~ 8850 2800
 Connection ~ 8950 2800
@@
 	9700 1900 10250 1900
 Wire Wire Line
-	10250 1850 10250 1950
+	10250 1850 10250 1900
+Wire Wire Line
+	10250 1900 10250 1950
 Connection ~ 10250 1900
 NoConn ~ 9700 2000
@@
 $EndComp
 Wire Wire Line
-	1450 4750 1750 4750
+	1450 4750 1650 4750
+Wire Wire Line
+	1650 4750 1750 4750
 Wire Wire Line
 	1650 4750 1650 4800
@@
 $EndComp
 Wire Wire Line
-	1450 5400 1750 5400
+	1450 5400 1650 5400
+Wire Wire Line
+	1650 5400 1750 5400
 Wire Wire Line
 	1650 5400 1650 5450

Commit message: Replace mag/accel and add addresses
Replace the mag/accel chip with one that is in stock and add all i2c device addresses as notes for reference
Parts:
- removed JP?: Jumper_NC_Small, symbol Jumper_NC_Small
- removed JP?: Jumper_NO_Small, symbol Jumper_NO_Small
- removed U?: LSM303DTR, symbol LSM303DTR
- added U?: LSM303DLHCTR, symbol LSM303DLHCTR
Connections:
- wire segments 99 -> 67
- no-connect marks 8 -> 6
Other:
- note added: "addr: 0x32"
- note added: "addr: 0x3C"
- note added: "addr: 0x70\n 0x72"
- note added: "addr: 0xD6 (alt 0xD4)"
- moved on the sheet: C?
Changed lines of the file:
@@
-$EndComp
-$Comp
-L LSM303DTR U?
-U 1 1 58759E44
-P 9000 2150
-F 0 "U?" H 9400 2600 60  0000 C CNN
-F 1 "LSM303DTR" H 9000 2150 60  0000 C CNB
-F 2 "" H 8250 2550 60  0001 C CNN
-F 3 "" H 8250 2550 60  0001 C CNN
-	1    9000 2150
-	1    0    0    -1
 $EndComp
 $Comp
@@
 L GND #PWR?
 U 1 1 58759E75
-P 8950 3200
-F 0 "#PWR?" H 8950 2950 50  0001 C CNN
-F 1 "GND" H 8950 3050 50  0001 C CNN
-F 2 "" H 8950 3200 50  0000 C CNN
-F 3 "" H 8950 3200 50  0000 C CNN
-	1    8950 3200
+P 8850 3200
+F 0 "#PWR?" H 8850 2950 50  0001 C CNN
+F 1 "GND" H 8850 3050 50  0001 C CNN
+F 2 "" H 8850 3200 50  0000 C CNN
+F 3 "" H 8850 3200 50  0000 C CNN
+	1    8850 3200
 	1    0    0    -1
 $EndComp
@@
 L C C?
 U 1 1 58759E7B
-P 9900 2250
-F 0 "C?" H 9925 2350 50  0000 L CNN
-F 1 "0.22uF" H 9925 2150 50  0000 L CNN
-F 2 "" H 9938 2100 50  0000 C CNN
-F 3 "" H 9900 2250 50  0000 C CNN
-	1    9900 2250
+P 10000 2250
+F 0 "C?" H 10025 2350 50  0000 L CNN
+F 1 "0.22uF" H 10025 2150 50  0000 L CNN
+F 2 "" H 10038 2100 50  0000 C CNN
+F 3 "" H 10000 2250 50  0000 C CNN
+	1    10000 2250
 	1    0    0    -1
 $EndComp
@@
 Connection ~ 3050 2900
 Wire Wire Line
-	2650 2800 2700 2800
-Wire Wire Line
-	2700 2800 2750 2800
-Wire Wire Line
-	2650 2900 3050 2900
-Wire Wire Line
-	3050 2900 3100 2900
+	2650 2800 2750 2800
+Wire Wire Line
+	2650 2900 3100 2900
 Wire Wire Line
 	1600 1800 1600 1950
@@
 	5800 3200 5500 3200
 Wire Wire Line
-	5500 3200 5500 2800
-Wire Wire Line
-	4700 2800 5200 2800
-Wire Wire Line
-	5200 2800 5300 2800
-Wire Wire Line
-	5300 2800 5400 2800
-Wire Wire Line
-	5400 2800 5500 2800
-Wire Wire Line
-	5500 2800 5600 2800
-Wire Wire Line
-	5600 2800 5700 2800
+	5500 2800 5500 3200
+Wire Wire Line
+	4700 2800 5700 2800
 Connection ~ 5600 2800
 Connection ~ 5500 2800
@@
 Connection ~ 5300 2800
 Wire Wire Line
-	4700 1250 5400 1250
-Wire Wire Line
-	5400 1250 5750 1250
-Wire Wire Line
-	5750 1250 6000 1250
-Wire Wire Line
-	6000 1250 6250 1250
+	4700 1250 6250 1250
 Connection ~ 6000 1250
 Wire Wire Line
-	5400 1200 5400 1250
-Wire Wire Line
-	5400 1250 5400 1550
+	5400 1200 5400 1550
 Connection ~ 5400 1250
 Wire Wire Line
 	5400 1550 5500 1550
 Wire Wire Line
-	5750 1550 6000 1550
-Wire Wire Line
-	6000 1550 6250 1550
+	5750 1550 6250 1550
 Connection ~ 6000 1550
 Wire Wire Line
@@
 	6150 2100 6700 2100
 Wire Wire Line
-	6700 2050 6700 2100
-Wire Wire Line
-	6700 2100 6700 2150
+	6700 2050 6700 2150
 Connection ~ 6700 2100
 Wire Wire Line
@@
 	6700 2350 6700 2400
 Wire Wire Line
-	9300 1550 9550 1550
-Wire Wire Line
-	9550 1550 9800 1550
+	9300 1550 9800 1550
 Connection ~ 9550 1550
 Wire Wire Line
-	8250 1250 8950 1250
-Wire Wire Line
-	8950 1250 9300 1250
-Wire Wire Line
-	9300 1250 9550 1250
-Wire Wire Line
-	9550 1250 9800 1250
+	8950 1250 9800 1250
 Connection ~ 9550 1250
 Wire Wire Line
-	8950 1200 8950 1250
-Wire Wire Line
-	8950 1250 8950 1550
+	8950 1200 8950 1550
 Connection ~ 9300 1250
-Wire Wire Line
-	8950 1550 9050 1550
-Wire Wire Line
-	8350 2000 8250 2000
-Wire Wire Line
-	8250 2000 8250 1250
 Connection ~ 8950 1250
 Wire Wire Line
 	9550 1600 9550 1550
 Wire Wire Line
-	8250 2200 8350 2200
-Wire Wire Line
-	8350 2100 8250 2100
-Wire Wire Line
-	8750 2800 8850 2800
-Wire Wire Line
-	8850 2800 8950 2800
-Wire Wire Line
-	8950 2800 9050 2800
-Wire Wire Line
-	9050 2800 9150 2800
+	8750 2800 8950 2800
 Connection ~ 8850 2800
-Connection ~ 8950 2800
-Connection ~ 9050 2800
 Wire Wire Line
 	9250 3150 9250 3200
 Wire Wire Line
-	9250 3200 8950 3200
-Wire Wire Line
-	8950 3200 8950 2800
+	9250 3200 8850 3200
 Wire Wire Line
 	9250 2800 9250 2850
 Wire Wire Line
-	9700 2300 9750 2300
-Wire Wire Line
-	9750 2300 9750 2400
-Wire Wire Line
-	9750 2400 9900 2400
-Wire Wire Line
-	9900 2100 9750 2100
-Wire Wire Line
-	9750 2100 9750 2200
-Wire Wire Line
-	9750 2200 9700 2200
-$Comp
-L GND #PWR?
-U 1 1 58759EDF
-P 10250 2200
-F 0 "#PWR?" H 10250 1950 50  0001 C CNN
-F 1 "GND" H 10250 2050 50  0001 C CNN
-F 2 "" H 10250 2200 50  0000 C CNN
-F 3 "" H 10250 2200 50  0000 C CNN
-	1    10250 2200
-	1    0    0    -1
-$EndComp
-Wire Wire Line
-	9700 1900 10250 1900
-Wire Wire Line
-	10250 1850 10250 1900
-Wire Wire Line
-	10250 1900 10250 1950
-Connection ~ 10250 1900
-NoConn ~ 9700 2000
-NoConn ~ 9700 2100
+	9800 2300 9850 2300
+Wire Wire Line
+	9850 2300 9850 2400
+Wire Wire Line
+	9850 2400 10000 2400
+Wire Wire Line
+	10000 2100 9850 2100
+Wire Wire Line
+	9850 2100 9850 2200
+Wire Wire Line
+	9850 2200 9800 2200
 NoConn ~ 6150 2300
 NoConn ~ 6150 2200
@@
 	0    -1   -1   0
 $EndComp
-$Comp
-L Jumper_NC_Small JP?
-U 1 1 58759F01
-P 10250 1750
-F 0 "JP?" H 10250 1830 50  0000 C CNN
-F 1 "Jumper_NC_Small" H 10260 1690 50  0001 C CNN
-F 2 "" H 10250 1750 50  0000 C CNN
-F 3 "" H 10250 1750 50  0000 C CNN
-	1    10250 1750
-	0    -1   -1   0
-$EndComp
-$Comp
-L Jumper_NO_Small JP?
-U 1 1 58759F08
-P 10250 2050
-F 0 "JP?" H 10250 2130 50  0000 C CNN
-F 1 "Jumper_NO_Small" H 10260 1990 50  0001 C CNN
-F 2 "" H 10250 2050 50  0000 C CNN
-F 3 "" H 10250 2050 50  0000 C CNN
-	1    10250 2050
-	0    -1   -1   0
-$EndComp
-Wire Wire Line
-	10250 2200 10250 2150
-Wire Wire Line
-	10250 1600 10250 1650
 NoConn ~ 1600 1550
 NoConn ~ 1600 2950
@@
 $EndComp
 Wire Wire Line
-	1450 4750 1650 4750
-Wire Wire Line
-	1650 4750 1750 4750
+	1450 4750 1750 4750
 Wire Wire Line
 	1650 4750 1650 4800
@@
 $EndComp
 Wire Wire Line
-	1450 5400 1650 5400
-Wire Wire Line
-	1650 5400 1750 5400
+	1450 5400 1750 5400
 Wire Wire Line
 	1650 5400 1650 5450
@@
 +3.3V
 Text HLabel 8950 1200 1    60   Input ~ 12
-+3.3V
-Text HLabel 10250 1600 1    60   Input ~ 12
 +3.3V
 Text HLabel 6700 1800 1    60   Input ~ 12
@@
 Text HLabel 1450 5400 0    60   Input ~ 12
 front_bumper
+$Comp
+L LSM303DLHCTR U?
+U 1 1 586C66E2
+P 9000 2150
+F 0 "U?" H 9400 2600 60  0000 C CNN
+F 1 "LSM303DLHCTR" H 9000 2150 60  0000 C CNB
+F 2 "" H 8250 2550 60  0001 C CNN
+F 3 "" H 8250 2550 60  0001 C CNN
+	1    9000 2150
+	1    0    0    -1
+$EndComp
+Wire Wire Line
+	8950 1550 9050 1550
+Wire Wire Line
+	8850 3200 8850 2800
+Text Notes 8250 600  0    60   ~ 0
+addr: 0x32
+Text Notes 8250 700  0    60   ~ 0
+addr: 0x3C
+Text Notes 4550 600  0    60   ~ 0
+addr: 0xD6 (alt 0xD4)
+Text Notes 1350 700  0    60   ~ 0
+addr: 0x70\n      0x72
 $EndSCHEMATC

Commit message: Fix errors in schematic
- Fix motor feedback circuit
- Replace micro SD card with standard symbol
- Replace some 0ohm's with cuttable traces
- Clean up motor sheet
Connections:
- wire segments 67 -> 65
Changed lines of the file:
@@
 EESchema Schematic File Version 2
 LIBS:PiBot-rescue
+LIBS:power
+LIBS:device
+LIBS:transistors
+LIBS:conn
+LIBS:linear
+LIBS:regul
+LIBS:74xx
+LIBS:cmos4000
+LIBS:adc-dac
+LIBS:memory
+LIBS:xilinx
+LIBS:microcontrollers
+LIBS:dsp
+LIBS:microchip
+LIBS:analog_switches
+LIBS:motorola
+LIBS:texas
+LIBS:intel
+LIBS:audio
+LIBS:interface
+LIBS:digital-audio
+LIBS:philips
+LIBS:display
+LIBS:cypress
+LIBS:siliconi
+LIBS:opto
+LIBS:atmel
+LIBS:contrib
+LIBS:valves
 LIBS:PiBot
+LIBS:74xgxx
+LIBS:ac-dc
+LIBS:actel
+LIBS:allegro
+LIBS:Altera
+LIBS:analog_devices
+LIBS:battery_management
+LIBS:bbd
+LIBS:bosch
+LIBS:brooktre
+LIBS:cmos_ieee
+LIBS:dc-dc
+LIBS:diode
+LIBS:elec-unifil
+LIBS:ESD_Protection
+LIBS:ftdi
+LIBS:gennum
+LIBS:graphic
+LIBS:hc11
+LIBS:ir
+LIBS:Lattice
+LIBS:logo
+LIBS:maxim
+LIBS:mechanical
+LIBS:microchip_dspic33dsc
+LIBS:microchip_pic10mcu
+LIBS:microchip_pic12mcu
+LIBS:microchip_pic16mcu
+LIBS:microchip_pic18mcu
+LIBS:microchip_pic32mcu
+LIBS:motor_drivers
+LIBS:motors
+LIBS:msp430
+LIBS:nordicsemi
+LIBS:nxp_armmcu
+LIBS:onsemi
+LIBS:Oscillators
+LIBS:powerint
+LIBS:Power_Management
+LIBS:pspice
+LIBS:references
+LIBS:relays
+LIBS:rfcom
+LIBS:sensors
+LIBS:silabs
+LIBS:stm8
+LIBS:stm32
+LIBS:supertex
+LIBS:switches
+LIBS:transf
+LIBS:ttl_ieee
+LIBS:video
+LIBS:wiznet
+LIBS:Worldsemi
+LIBS:Xicor
+LIBS:zetex
+LIBS:Zilog
 LIBS:PiBot-cache
 EELAYER 25 0
@@
 	5800 3200 5500 3200
 Wire Wire Line
-	5500 2800 5500 3200
+	5500 3200 5500 2800
 Wire Wire Line
 	4700 2800 5700 2800
@@
 L GND #PWR?
 U 1 1 5875CDBA
-P 3000 4950
-F 0 "#PWR?" H 3000 4700 50  0001 C CNN
-F 1 "GND" H 2950 4800 50  0001 C CNN
-F 2 "" H 3000 4950 50  0000 C CNN
-F 3 "" H 3000 4950 50  0000 C CNN
-	1    3000 4950
-	1    0    0    -1
-$EndComp
-Wire Wire Line
-	2550 4850 2650 4850
-Wire Wire Line
-	2550 4650 2650 4650
+P 2150 5150
+F 0 "#PWR?" H 2150 4900 50  0001 C CNN
+F 1 "GND" H 2100 5000 50  0001 C CNN
+F 2 "" H 2150 5150 50  0000 C CNN
+F 3 "" H 2150 5150 50  0000 C CNN
+	1    2150 5150
+	1    0    0    -1
+$EndComp
 $Comp
 L C C?
@@
 L R R?
 U 1 1 5875CDD2
-P 2800 4850
-F 0 "R?" V 2880 4850 50  0000 C CNN
-F 1 "10k" V 2800 4850 50  0000 C CNN
-F 2 "" V 2730 4850 50  0000 C CNN
-F 3 "" H 2800 4850 50  0000 C CNN
-	1    2800 4850
-	0    1    1    0
-$EndComp
-Wire Wire Line
-	2950 4850 3000 4850
-Wire Wire Line
-	3000 4850 3000 4950
+P 2150 4950
+F 0 "R?" V 2230 4950 50  0000 C CNN
+F 1 "10k" V 2150 4950 50  0000 C CNN
+F 2 "" V 2080 4950 50  0000 C CNN
+F 3 "" H 2150 4950 50  0000 C CNN
+	1    2150 4950
+	-1   0    0    1
+$EndComp
 $Comp
 L R R?
@@
 L GND #PWR?
 U 1 1 5875CDF5
-P 3000 5600
-F 0 "#PWR?" H 3000 5350 50  0001 C CNN
-F 1 "GND" H 2950 5450 50  0001 C CNN
-F 2 "" H 3000 5600 50  0000 C CNN
-F 3 "" H 3000 5600 50  0000 C CNN
-	1    3000 5600
-	1    0    0    -1
-$EndComp
-Wire Wire Line
-	2550 5500 2650 5500
-Wire Wire Line
-	2550 5300 2650 5300
+P 2150 5800
+F 0 "#PWR?" H 2150 5550 50  0001 C CNN
+F 1 "GND" H 2100 5650 50  0001 C CNN
+F 2 "" H 2150 5800 50  0000 C CNN
+F 3 "" H 2150 5800 50  0000 C CNN
+	1    2150 5800
+	1    0    0    -1
+$EndComp
 $Comp
 L C C?
@@
 L R R?
 U 1 1 5875CE0B
-P 2800 5500
-F 0 "R?" V 2880 5500 50  0000 C CNN
-F 1 "10k" V 2800 5500 50  0000 C CNN
-F 2 "" V 2730 5500 50  0000 C CNN
-F 3 "" H 2800 5500 50  0000 C CNN
-	1    2800 5500
-	0    1    1    0
-$EndComp
-Wire Wire Line
-	2950 5500 3000 5500
-Wire Wire Line
-	3000 5500 3000 5600
+P 2150 5600
+F 0 "R?" V 2230 5600 50  0000 C CNN
+F 1 "10k" V 2150 5600 50  0000 C CNN
+F 2 "" V 2080 5600 50  0000 C CNN
+F 3 "" H 2150 5600 50  0000 C CNN
+	1    2150 5600
+	-1   0    0    1
+$EndComp
 $Comp
 L R R?
@@
 Text Notes 550  3950 0    60   ~ 12
 Bumpers
-Text HLabel 2650 4650 2    60   Input ~ 12
+Text HLabel 2650 4850 2    60   Input ~ 12
 +3.3V
-Text HLabel 2650 5300 2    60   Input ~ 12
+Text HLabel 2650 5500 2    60   Input ~ 12
 +3.3V
 Text HLabel 1600 2750 1    60   Input ~ 12
@@
 Text Notes 1350 700  0    60   ~ 0
 addr: 0x70\n      0x72
+Wire Wire Line
+	2150 5150 2150 5100
+Wire Wire Line
+	2150 4750 2150 4800
+Wire Wire Line
+	2150 5400 2150 5450
+Wire Wire Line
+	2150 5800 2150 5750
+Wire Wire Line
+	2650 5500 2550 5500
+Wire Wire Line
+	2650 4850 2550 4850
 $EndSCHEMATC

Commit message: Minor cleanup
Other:
- note added: "By:\nBroderick Carlin\nTyler Holmes"
- note added: "MIT License\n"
- note added: "PycoBot (Teensy uPython Robot)"
Changed lines of the file:
@@
 Wire Wire Line
 	2650 4850 2550 4850
+Text Notes 7050 7050 0    60   ~ 12
+By:\nBroderick Carlin\nTyler Holmes
+Text Notes 7950 7050 0    60   ~ 12
+MIT License\n
+Text Notes 7350 7500 0    60   ~ 12
+PycoBot (Teensy uPython Robot)
 $EndSCHEMATC

Commit message: Fix some errors and add test point
Fixed errors with motor pinout and add test points
Parts:
- removed W? (x2): TP, symbol TEST_1P
- added SW? (x2): SW_SPDT, symbol SW_SPDT
Connections:
- wire segments 65 -> 67
Other:
- note added: "front left"
- note added: "front right"
- note added: "rear left"
- note added: "rear right"
- moved on the sheet: C?
Changed lines of the file:
@@
-$EndComp
-$Comp
-L TEST_1P W?
-U 1 1 58759DE5
-P 2700 2800
-F 0 "W?" H 2600 3050 50  0000 L TNN
-F 1 "TP" H 2550 2950 50  0000 L CNN
-F 2 "" H 2900 2800 50  0000 C CNN
-F 3 "" H 2900 2800 50  0000 C CNN
-	1    2700 2800
-	1    0    0    -1
-$EndComp
-$Comp
-L TEST_1P W?
-U 1 1 58759DEC
-P 3050 2900
-F 0 "W?" H 3050 3150 50  0000 L TNN
-F 1 "TP" H 3100 3050 50  0000 L CNN
-F 2 "" H 3250 2900 50  0000 C CNN
-F 3 "" H 3250 2900 50  0000 C CNN
-	1    3050 2900
-	1    0    0    -1
 $EndComp
 $Comp
@@
 	1    0    0    -1
 $EndComp
-Connection ~ 2700 2800
 Connection ~ 3050 2900
-Wire Wire Line
-	2650 2800 2750 2800
 Wire Wire Line
 	2650 2900 3100 2900
@@
 L SW_SPDT SW?
 U 1 1 5875CDB3
-P 2350 4750
-F 0 "SW?" H 2350 4920 50  0000 C CNN
-F 1 "SW_SPDT" H 2350 4550 50  0001 C CNN
-F 2 "" H 2350 4750 50  0000 C CNN
-F 3 "" H 2350 4750 50  0000 C CNN
-	1    2350 4750
+P 2350 4400
+F 0 "SW?" H 2350 4570 50  0000 C CNN
+F 1 "SW_SPDT" H 2350 4200 50  0001 C CNN
+F 2 "" H 2350 4400 50  0000 C CNN
+F 3 "" H 2350 4400 50  0000 C CNN
+	1    2350 4400
 	1    0    0    -1
 $EndComp
@@
 L GND #PWR?
 U 1 1 5875CDBA
-P 2150 5150
-F 0 "#PWR?" H 2150 4900 50  0001 C CNN
-F 1 "GND" H 2100 5000 50  0001 C CNN
-F 2 "" H 2150 5150 50  0000 C CNN
-F 3 "" H 2150 5150 50  0000 C CNN
-	1    2150 5150
+P 2150 4800
+F 0 "#PWR?" H 2150 4550 50  0001 C CNN
+F 1 "GND" H 2100 4650 50  0001 C CNN
+F 2 "" H 2150 4800 50  0000 C CNN
+F 3 "" H 2150 4800 50  0000 C CNN
+	1    2150 4800
 	1    0    0    -1
 $EndComp
@@
 L C C?
 U 1 1 5875CDCB
-P 1650 4950
-F 0 "C?" H 1675 5050 50  0000 L CNN
-F 1 "0.1uF" H 1675 4850 50  0000 L CNN
-F 2 "" H 1688 4800 50  0000 C CNN
-F 3 "" H 1650 4950 50  0000 C CNN
-	1    1650 4950
+P 1650 4600
+F 0 "C?" H 1675 4700 50  0000 L CNN
+F 1 "0.1uF" H 1675 4500 50  0000 L CNN
+F 2 "" H 1688 4450 50  0000 C CNN
+F 3 "" H 1650 4600 50  0000 C CNN
+	1    1650 4600
 	1    0    0    -1
 $EndComp
@@
 L R R?
 U 1 1 5875CDD2
-P 2150 4950
-F 0 "R?" V 2230 4950 50  0000 C CNN
-F 1 "10k" V 2150 4950 50  0000 C CNN
-F 2 "" V 2080 4950 50  0000 C CNN
-F 3 "" H 2150 4950 50  0000 C CNN
-	1    2150 4950
+P 2150 4600
+F 0 "R?" V 2230 4600 50  0000 C CNN
+F 1 "10k" V 2150 4600 50  0000 C CNN
+F 2 "" V 2080 4600 50  0000 C CNN
+F 3 "" H 2150 4600 50  0000 C CNN
+	1    2150 4600
 	-1   0    0    1
 $EndComp
@@
 L R R?
 U 1 1 5875CDDB
-P 1900 4750
-F 0 "R?" V 1980 4750 50  0000 C CNN
-F 1 "10k" V 1900 4750 50  0000 C CNN
-F 2 "" V 1830 4750 50  0000 C CNN
-F 3 "" H 1900 4750 50  0000 C CNN
-	1    1900 4750
+P 1900 4400
+F 0 "R?" V 1980 4400 50  0000 C CNN
+F 1 "10k" V 1900 4400 50  0000 C CNN
+F 2 "" V 1830 4400 50  0000 C CNN
+F 3 "" H 1900 4400 50  0000 C CNN
+	1    1900 4400
 	0    1    1    0
 $EndComp
 Wire Wire Line
-	1450 4750 1750 4750
-Wire Wire Line
-	1650 4750 1650 4800
-Connection ~ 1650 4750
-Wire Wire Line
-	2050 4750 2150 4750
+	1450 4400 1750 4400
+Wire Wire Line
+	1650 4400 1650 4450
+Connection ~ 1650 4400
+Wire Wire Line
+	2050 4400 2150 4400
 $Comp
 L GND #PWR?
 U 1 1 5875CDE7
-P 1650 5150
-F 0 "#PWR?" H 1650 4900 50  0001 C CNN
-F 1 "GND" H 1600 5000 50  0001 C CNN
-F 2 "" H 1650 5150 50  0000 C CNN
-F 3 "" H 1650 5150 50  0000 C CNN
-	1    1650 5150
-	1    0    0    -1
-$EndComp
-Wire Wire Line
-	1650 5150 1650 5100
+P 1650 4800
+F 0 "#PWR?" H 1650 4550 50  0001 C CNN
+F 1 "GND" H 1600 4650 50  0001 C CNN
+F 2 "" H 1650 4800 50  0000 C CNN
+F 3 "" H 1650 4800 50  0000 C CNN
+	1    1650 4800
+	1    0    0    -1
+$EndComp
+Wire Wire Line
+	1650 4800 1650 4750
 $Comp
 L SW_SPDT SW?
@@
 Text Notes 550  3950 0    60   ~ 12
 Bumpers
-Text HLabel 2650 4850 2    60   Input ~ 12
+Text HLabel 2650 4500 2    60   Input ~ 12
 +3.3V
 Text HLabel 2650 5500 2    60   Input ~ 12
@@
 NoConn ~ 2650 3200
 NoConn ~ 2650 1800
-Text HLabel 1450 4750 0    60   Input ~ 12
+Text HLabel 1450 4400 0    60   Input ~ 12
 rear_bumper
 Text HLabel 1450 5400 0    60   Input ~ 12
@@
 addr: 0x70\n      0x72
 Wire Wire Line
-	2150 5150 2150 5100
-Wire Wire Line
-	2150 4750 2150 4800
-Wire Wire Line
-	2150 5400 2150 5450
+	2150 4800 2150 4750
+Wire Wire Line
+	2150 4050 2150 4450
+Wire Wire Line
+	2150 5050 2150 5450
 Wire Wire Line
 	2150 5800 2150 5750
@@
 	2650 5500 2550 5500
 Wire Wire Line
-	2650 4850 2550 4850
+	2650 4500 2550 4500
 Text Notes 7050 7050 0    60   ~ 12
 By:\nBroderick Carlin\nTyler Holmes
@@
 Text Notes 7350 7500 0    60   ~ 12
 PycoBot (Teensy uPython Robot)
+$Comp
+L SW_SPDT SW?
+U 1 1 586E605E
+P 2350 4050
+F 0 "SW?" H 2350 4220 50  0000 C CNN
+F 1 "SW_SPDT" H 2350 3850 50  0001 C CNN
+F 2 "" H 2350 4050 50  0000 C CNN
+F 3 "" H 2350 4050 50  0000 C CNN
+	1    2350 4050
+	1    0    0    -1
+$EndComp
+Text HLabel 2650 4150 2    60   Input ~ 12
++3.3V
+Wire Wire Line
+	2650 4150 2550 4150
+Connection ~ 2150 4400
+$Comp
+L SW_SPDT SW?
+U 1 1 586E63D0
+P 2350 5050
+F 0 "SW?" H 2350 5220 50  0000 C CNN
+F 1 "SW_SPDT" H 2350 4850 50  0001 C CNN
+F 2 "" H 2350 5050 50  0000 C CNN
+F 3 "" H 2350 5050 50  0000 C CNN
+	1    2350 5050
+	1    0    0    -1
+$EndComp
+Text HLabel 2650 5150 2    60   Input ~ 12
++3.3V
+Wire Wire Line
+	2650 5150 2550 5150
+Connection ~ 2150 5400
+Text Notes 3100 4050 0    60   ~ 0
+rear left
+Text Notes 3100 4450 0    60   ~ 0
+rear right
+Text Notes 3100 5050 0    60   ~ 0
+front left
+Text Notes 3100 5450 0    60   ~ 0
+front right
+Wire Wire Line
+	2650 2800 2750 2800
 $EndSCHEMATC
