File: hardware/KiCAD/sensors.sch (KiCad schematic (older format))
At the start: 31 parts

Commit message: Add MacroFab library and update SD card
Parts:
- C36, C37, C38, C39, C41, C42, C43, C46, C47: renamed from C?; footprint (none) -> Capacitors_SMD:C_0402
- C40, C45: renamed from C?; footprint (none) -> Capacitors_SMD:C_1206
- C44, C48: renamed from C?; footprint (none) -> Resistors_SMD:R_0402
- P10, P9: renamed from P?; footprint (none) -> Pin_Headers:Pin_Header_Straight_1x01_Pitch2.54mm
- P11: renamed from P?; footprint (none) -> Pin_Headers:Pin_Header_Straight_2x01_Pitch2.54mm
- P12: renamed from P?; footprint (none) -> Pin_Headers:Pin_Header_Straight_1x03_Pitch2.54mm
- R28, R29, R30, R31: renamed from R?; footprint (none) -> Resistors_SMD:R_0402
- U13, U14: renamed from U?; footprint PiBot:WSON008X2120 -> (none)
- gave numbers to parts that had none: 8
