File: hardware/KiCAD/sensors.sch (KiCad schematic (older format))
At the start: 31 parts, among them P10 BREAKOUT, P11 BREAKOUT, P12 BREAKOUT, P9 BREAKOUT, SW2 SW_SPDT, SW3 SW_SPDT, SW4 SW_SPDT, SW5 SW_SPDT, U13 BH1745NUC, U14 BH1745NUC, U15 L3GD20H, U16 LSM303DLHCTR

Commit message: Add the rest of the missing footprints, aside from motor
Parts:
- JP15: footprint (none) -> PiBot:Jumper-NC
- JP16: footprint (none) -> PiBot:Jumper-NO
- SW2, SW3, SW4, SW5: footprint (none) -> PiBot:TS0101F020V3; Part Number (none) -> TS0101F020V3
Changed lines of the file:
@@
 $EndComp
 $Comp
-L GND #PWR078
+L GND #PWR056
 U 1 1 58759DD1
 P 1600 3350
-F 0 "#PWR078" H 1600 3100 50  0001 C CNN
+F 0 "#PWR056" H 1600 3100 50  0001 C CNN
 F 1 "GND" H 1600 3200 50  0001 C CNN
 F 2 "" H 1600 3350 50  0000 C CNN
@@
 $EndComp
 $Comp
-L GND #PWR079
+L GND #PWR057
 U 1 1 58759DD7
 P 2650 3350
-F 0 "#PWR079" H 2650 3100 50  0001 C CNN
+F 0 "#PWR057" H 2650 3100 50  0001 C CNN
 F 1 "GND" H 2650 3200 50  0001 C CNN
 F 2 "" H 2650 3350 50  0000 C CNN
@@
 $EndComp
 $Comp
-L GND #PWR080
+L GND #PWR058
 U 1 1 58759DDD
 P 1600 1950
-F 0 "#PWR080" H 1600 1700 50  0001 C CNN
+F 0 "#PWR058" H 1600 1700 50  0001 C CNN
 F 1 "GND" H 1600 1800 50  0001 C CNN
 F 2 "" H 1600 1950 50  0000 C CNN
@@
 $EndComp
 $Comp
-L GND #PWR081
+L GND #PWR059
 U 1 1 58759E0F
 P 5800 3200
-F 0 "#PWR081" H 5800 2950 50  0001 C CNN
+F 0 "#PWR059" H 5800 2950 50  0001 C CNN
 F 1 "GND" H 5800 3050 50  0001 C CNN
 F 2 "" H 5800 3200 50  0000 C CNN
@@
 $EndComp
 $Comp
-L GND #PWR082
+L GND #PWR060
 U 1 1 58759E22
 P 6000 1600
-F 0 "#PWR082" H 6000 1350 50  0001 C CNN
+F 0 "#PWR060" H 6000 1350 50  0001 C CNN
 F 1 "GND" H 6000 1450 50  0001 C CNN
 F 2 "" H 6000 1600 50  0000 C CNN
@@
 $EndComp
 $Comp
-L GND #PWR083
+L GND #PWR061
 U 1 1 58759E38
 P 6700 2400
-F 0 "#PWR083" H 6700 2150 50  0001 C CNN
+F 0 "#PWR061" H 6700 2150 50  0001 C CNN
 F 1 "GND" H 6700 2250 50  0001 C CNN
 F 2 "" H 6700 2400 50  0000 C CNN
@@
 $EndComp
 $Comp
-L GND #PWR084
+L GND #PWR062
 U 1 1 58759E66
 P 9550 1600
-F 0 "#PWR084" H 9550 1350 50  0001 C CNN
+F 0 "#PWR062" H 9550 1350 50  0001 C CNN
 F 1 "GND" H 9550 1450 50  0001 C CNN
 F 2 "" H 9550 1600 50  0000 C CNN
@@
 $EndComp
 $Comp
-L GND #PWR085
+L GND #PWR063
 U 1 1 58759E75
 P 8850 3200
-F 0 "#PWR085" H 8850 2950 50  0001 C CNN
+F 0 "#PWR063" H 8850 2950 50  0001 C CNN
 F 1 "GND" H 8850 3050 50  0001 C CNN
 F 2 "" H 8850 3200 50  0000 C CNN
@@
 F 0 "JP15" H 6700 2030 50  0000 C CNN
 F 1 "Jumper_NC_Small" H 6710 1890 50  0001 C CNN
-F 2 "" H 6700 1950 50  0001 C CNN
+F 2 "PiBot:Jumper-NC" H 6700 1950 50  0001 C CNN
 F 3 "" H 6700 1950 50  0000 C CNN
 	1    6700 1950
@@
 F 0 "JP16" H 6700 2330 50  0000 C CNN
 F 1 "Jumper_NO_Small" H 6710 2190 50  0001 C CNN
-F 2 "" H 6700 2250 50  0001 C CNN
+F 2 "PiBot:Jumper-NO" H 6700 2250 50  0001 C CNN
 F 3 "" H 6700 2250 50  0000 C CNN
 	1    6700 2250
@@
 Color Sensors
 $Comp
-L SW_SPDT SW3
-U 1 1 5875CDB3
-P 2350 4400
-F 0 "SW3" H 2350 4570 50  0000 C CNN
-F 1 "SW_SPDT" H 2350 4200 50  0001 C CNN
-F 2 "" H 2350 4400 50  0001 C CNN
-F 3 "" H 2350 4400 50  0000 C CNN
-	1    2350 4400
-	1    0    0    -1
-$EndComp
-$Comp
-L GND #PWR086
+L GND #PWR064
 U 1 1 5875CDBA
 P 2150 4800
-F 0 "#PWR086" H 2150 4550 50  0001 C CNN
+F 0 "#PWR064" H 2150 4550 50  0001 C CNN
 F 1 "GND" H 2100 4650 50  0001 C CNN
 F 2 "" H 2150 4800 50  0000 C CNN
@@
 	2050 4400 2150 4400
 $Comp
-L GND #PWR087
+L GND #PWR065
 U 1 1 5875CDE7
 P 1650 4800
-F 0 "#PWR087" H 1650 4550 50  0001 C CNN
+F 0 "#PWR065" H 1650 4550 50  0001 C CNN
 F 1 "GND" H 1600 4650 50  0001 C CNN
 F 2 "" H 1650 4800 50  0000 C CNN
@@
 	1650 4800 1650 4750
 $Comp
-L SW_SPDT SW5
-U 1 1 5875CDEE
-P 2350 5400
-F 0 "SW5" H 2350 5570 50  0000 C CNN
-F 1 "SW_SPDT" H 2350 5200 50  0001 C CNN
-F 2 "" H 2350 5400 50  0001 C CNN
-F 3 "" H 2350 5400 50  0000 C CNN
-	1    2350 5400
-	1    0    0    -1
-$EndComp
-$Comp
-L GND #PWR088
+L GND #PWR066
 U 1 1 5875CDF5
 P 2150 5800
-F 0 "#PWR088" H 2150 5550 50  0001 C CNN
+F 0 "#PWR066" H 2150 5550 50  0001 C CNN
 F 1 "GND" H 2100 5650 50  0001 C CNN
 F 2 "" H 2150 5800 50  0000 C CNN
@@
 	2050 5400 2150 5400
 $Comp
-L GND #PWR089
+L GND #PWR067
 U 1 1 5875CE20
 P 1650 5800
-F 0 "#PWR089" H 1650 5550 50  0001 C CNN
+F 0 "#PWR067" H 1650 5550 50  0001 C CNN
 F 1 "GND" H 1600 5650 50  0001 C CNN
 F 2 "" H 1650 5800 50  0000 C CNN
@@
 F 0 "SW2" H 2350 4220 50  0000 C CNN
 F 1 "SW_SPDT" H 2350 3850 50  0001 C CNN
-F 2 "" H 2350 4050 50  0001 C CNN
+F 2 "PiBot:TS0101F020V3" H 2350 4050 50  0001 C CNN
 F 3 "" H 2350 4050 50  0000 C CNN
+F 4 "TS0101F020V3" H 2350 4050 60  0001 C CNN "Part Number"
 	1    2350 4050
 	1    0    0    -1
@@
 	2650 4150 2550 4150
 Connection ~ 2150 4400
-$Comp
-L SW_SPDT SW4
-U 1 1 586E63D0
-P 2350 5050
-F 0 "SW4" H 2350 5220 50  0000 C CNN
-F 1 "SW_SPDT" H 2350 4850 50  0001 C CNN
-F 2 "" H 2350 5050 50  0001 C CNN
-F 3 "" H 2350 5050 50  0000 C CNN
-	1    2350 5050
-	1    0    0    -1
-$EndComp
 Text HLabel 2650 5150 2    60   Input ~ 12
 +3.3V
@@
 	1    0    0    -1
 $EndComp
+$Comp
+L SW_SPDT SW3
+U 1 1 587817F7
+P 2350 4400
+F 0 "SW3" H 2350 4570 50  0000 C CNN
+F 1 "SW_SPDT" H 2350 4200 50  0001 C CNN
+F 2 "PiBot:TS0101F020V3" H 2350 4400 50  0001 C CNN
+F 3 "" H 2350 4400 50  0000 C CNN
+F 4 "TS0101F020V3" H 2350 4400 60  0001 C CNN "Part Number"
+	1    2350 4400
+	1    0    0    -1
+$EndComp
+$Comp
+L SW_SPDT SW4
+U 1 1 5878186E
+P 2350 5050
+F 0 "SW4" H 2350 5220 50  0000 C CNN
+F 1 "SW_SPDT" H 2350 4850 50  0001 C CNN
+F 2 "PiBot:TS0101F020V3" H 2350 5050 50  0001 C CNN
+F 3 "" H 2350 5050 50  0000 C CNN
+F 4 "TS0101F020V3" H 2350 5050 60  0001 C CNN "Part Number"
+	1    2350 5050
+	1    0    0    -1
+$EndComp
+$Comp
+L SW_SPDT SW5
+U 1 1 587818F0
+P 2350 5400
+F 0 "SW5" H 2350 5570 50  0000 C CNN
+F 1 "SW_SPDT" H 2350 5200 50  0001 C CNN
+F 2 "PiBot:TS0101F020V3" H 2350 5400 50  0001 C CNN
+F 3 "" H 2350 5400 50  0000 C CNN
+F 4 "TS0101F020V3" H 2350 5400 60  0001 C CNN "Part Number"
+	1    2350 5400
+	1    0    0    -1
+$EndComp

Commit message: Headway on schematic layout
Parts:
- removed P10, P9: BREAKOUT, Pin_Headers:Pin_Header_Straight_1x01_Pitch2.54mm, symbol CONN_01X01
- removed P11: BREAKOUT, Pin_Headers:Pin_Header_Straight_2x01_Pitch2.54mm, symbol CONN_01X02
- removed P12: BREAKOUT, Pin_Headers:Pin_Header_Straight_1x03_Pitch2.54mm, symbol CONN_01X03
- added DRDY1, INT1, INT2, TP10, TP12, TP4, TP6: TEST, Measurement_Points:Measurement_Point_Round-SMD-Pad_Small, symbol TEST
Changed lines of the file:
@@
 $EndComp
 $Comp
-L GND #PWR056
+L GND #PWR2
 U 1 1 58759DD1
 P 1600 3350
-F 0 "#PWR056" H 1600 3100 50  0001 C CNN
+F 0 "#PWR2" H 1600 3100 50  0001 C CNN
 F 1 "GND" H 1600 3200 50  0001 C CNN
 F 2 "" H 1600 3350 50  0000 C CNN
@@
 $EndComp
 $Comp
-L GND #PWR057
+L GND #PWR7
 U 1 1 58759DD7
 P 2650 3350
-F 0 "#PWR057" H 2650 3100 50  0001 C CNN
+F 0 "#PWR7" H 2650 3100 50  0001 C CNN
 F 1 "GND" H 2650 3200 50  0001 C CNN
 F 2 "" H 2650 3350 50  0000 C CNN
@@
 $EndComp
 $Comp
-L GND #PWR058
+L GND #PWR1
 U 1 1 58759DDD
 P 1600 1950
-F 0 "#PWR058" H 1600 1700 50  0001 C CNN
+F 0 "#PWR1" H 1600 1700 50  0001 C CNN
 F 1 "GND" H 1600 1800 50  0001 C CNN
 F 2 "" H 1600 1950 50  0000 C CNN
@@
 $EndComp
 $Comp
-L GND #PWR059
+L GND #PWR8
 U 1 1 58759E0F
 P 5800 3200
-F 0 "#PWR059" H 5800 2950 50  0001 C CNN
+F 0 "#PWR8" H 5800 2950 50  0001 C CNN
 F 1 "GND" H 5800 3050 50  0001 C CNN
 F 2 "" H 5800 3200 50  0000 C CNN
@@
 $EndComp
 $Comp
-L GND #PWR060
+L GND #PWR9
 U 1 1 58759E22
 P 6000 1600
-F 0 "#PWR060" H 6000 1350 50  0001 C CNN
+F 0 "#PWR9" H 6000 1350 50  0001 C CNN
 F 1 "GND" H 6000 1450 50  0001 C CNN
 F 2 "" H 6000 1600 50  0000 C CNN
@@
 $EndComp
 $Comp
-L GND #PWR061
+L GND #PWR10
 U 1 1 58759E38
 P 6700 2400
-F 0 "#PWR061" H 6700 2150 50  0001 C CNN
+F 0 "#PWR10" H 6700 2150 50  0001 C CNN
 F 1 "GND" H 6700 2250 50  0001 C CNN
 F 2 "" H 6700 2400 50  0000 C CNN
@@
 $EndComp
 $Comp
-L GND #PWR062
+L GND #PWR12
 U 1 1 58759E66
 P 9550 1600
-F 0 "#PWR062" H 9550 1350 50  0001 C CNN
+F 0 "#PWR12" H 9550 1350 50  0001 C CNN
 F 1 "GND" H 9550 1450 50  0001 C CNN
 F 2 "" H 9550 1600 50  0000 C CNN
@@
 $EndComp
 $Comp
-L GND #PWR063
+L GND #PWR11
 U 1 1 58759E75
 P 8850 3200
-F 0 "#PWR063" H 8850 2950 50  0001 C CNN
+F 0 "#PWR11" H 8850 2950 50  0001 C CNN
 F 1 "GND" H 8850 3050 50  0001 C CNN
 F 2 "" H 8850 3200 50  0000 C CNN
@@
 Color Sensors
 $Comp
-L GND #PWR064
+L GND #PWR5
 U 1 1 5875CDBA
 P 2150 4800
-F 0 "#PWR064" H 2150 4550 50  0001 C CNN
+F 0 "#PWR5" H 2150 4550 50  0001 C CNN
 F 1 "GND" H 2100 4650 50  0001 C CNN
 F 2 "" H 2150 4800 50  0000 C CNN
@@
 	2050 4400 2150 4400
 $Comp
-L GND #PWR065
+L GND #PWR3
 U 1 1 5875CDE7
 P 1650 4800
-F 0 "#PWR065" H 1650 4550 50  0001 C CNN
+F 0 "#PWR3" H 1650 4550 50  0001 C CNN
 F 1 "GND" H 1600 4650 50  0001 C CNN
 F 2 "" H 1650 4800 50  0000 C CNN
@@
 	1650 4800 1650 4750
 $Comp
-L GND #PWR066
+L GND #PWR6
 U 1 1 5875CDF5
 P 2150 5800
-F 0 "#PWR066" H 2150 5550 50  0001 C CNN
+F 0 "#PWR6" H 2150 5550 50  0001 C CNN
 F 1 "GND" H 2100 5650 50  0001 C CNN
 F 2 "" H 2150 5800 50  0000 C CNN
@@
 	2050 5400 2150 5400
 $Comp
-L GND #PWR067
+L GND #PWR4
 U 1 1 5875CE20
 P 1650 5800
-F 0 "#PWR067" H 1650 5550 50  0001 C CNN
+F 0 "#PWR4" H 1650 5550 50  0001 C CNN
 F 1 "GND" H 1600 5650 50  0001 C CNN
 F 2 "" H 1650 5800 50  0000 C CNN
@@
 Per datasheet,\nconnect reserved\npins to GND.
 $Comp
-L CONN_01X01 P9
-U 1 1 586DD209
-P 2850 1800
-F 0 "P9" H 2928 1841 50  0000 L CNN
-F 1 "BREAKOUT" H 2928 1750 50  0000 L CNN
-F 2 "Pin_Headers:Pin_Header_Straight_1x01_Pitch2.54mm" H 2850 1800 50  0001 C CNN
-F 3 "" H 2850 1800 50  0000 C CNN
-	1    2850 1800
-	1    0    0    -1
-$EndComp
-$Comp
-L CONN_01X01 P10
-U 1 1 586DD2E1
-P 2850 3200
-F 0 "P10" H 2928 3241 50  0000 L CNN
-F 1 "BREAKOUT" H 2928 3150 50  0000 L CNN
-F 2 "Pin_Headers:Pin_Header_Straight_1x01_Pitch2.54mm" H 2850 3200 50  0001 C CNN
-F 3 "" H 2850 3200 50  0000 C CNN
-	1    2850 3200
-	1    0    0    -1
-$EndComp
-$Comp
-L CONN_01X02 P11
-U 1 1 586DD782
-P 6350 2250
-F 0 "P11" H 6428 2291 50  0000 L CNN
-F 1 "BREAKOUT" H 6150 2100 50  0000 L CNN
-F 2 "Pin_Headers:Pin_Header_Straight_2x01_Pitch2.54mm" H 6350 2250 50  0001 C CNN
-F 3 "" H 6350 2250 50  0000 C CNN
-	1    6350 2250
-	1    0    0    -1
-$EndComp
-$Comp
-L CONN_01X03 P12
-U 1 1 586DDBFB
-P 10000 2000
-F 0 "P12" H 10078 2041 50  0000 L CNN
-F 1 "BREAKOUT" H 10078 1950 50  0000 L CNN
-F 2 "Pin_Headers:Pin_Header_Straight_1x03_Pitch2.54mm" H 10000 2000 50  0001 C CNN
-F 3 "" H 10000 2000 50  0000 C CNN
-	1    10000 2000
-	1    0    0    -1
-$EndComp
-$Comp
 L SW_SPDT SW3
 U 1 1 587817F7
@@
 	1    0    0    -1
 $EndComp
+$Comp
+L TEST DRDY1
+U 1 1 58E37DBB
+P 9800 1900
+F 0 "DRDY1" H 9800 2200 50  0000 C BNN
+F 1 "TEST" H 9800 2150 50  0000 C CNN
+F 2 "Measurement_Points:Measurement_Point_Round-SMD-Pad_Small" H 9800 1900 50  0001 C CNN
+F 3 "" H 9800 1900 50  0000 C CNN
+	1    9800 1900
+	0    1    1    0
+$EndComp
+$Comp
+L TEST INT1
+U 1 1 58E380BD
+P 9800 2000
+F 0 "INT1" H 9800 2300 50  0000 C BNN
+F 1 "TEST" H 9800 2250 50  0000 C CNN
+F 2 "Measurement_Points:Measurement_Point_Round-SMD-Pad_Small" H 9800 2000 50  0001 C CNN
+F 3 "" H 9800 2000 50  0000 C CNN
+	1    9800 2000
+	0    1    1    0
+$EndComp
+$Comp
+L TEST INT2
+U 1 1 58E3812E
+P 9800 2100
+F 0 "INT2" H 9800 2400 50  0000 C BNN
+F 1 "TEST" H 9800 2350 50  0000 C CNN
+F 2 "Measurement_Points:Measurement_Point_Round-SMD-Pad_Small" H 9800 2100 50  0001 C CNN
+F 3 "" H 9800 2100 50  0000 C CNN
+	1    9800 2100
+	0    1    1    0
+$EndComp
+$Comp
+L TEST TP10
+U 1 1 58E381F8
+P 6150 2200
+F 0 "TP10" H 6150 2500 50  0000 C BNN
+F 1 "TEST" H 6150 2450 50  0000 C CNN
+F 2 "Measurement_Points:Measurement_Point_Round-SMD-Pad_Small" H 6150 2200 50  0001 C CNN
+F 3 "" H 6150 2200 50  0000 C CNN
+	1    6150 2200
+	0    1    1    0
+$EndComp
+$Comp
+L TEST TP12
+U 1 1 58E384C9
+P 6150 2300
+F 0 "TP12" H 6150 2600 50  0000 C BNN
+F 1 "TEST" H 6150 2550 50  0000 C CNN
+F 2 "Measurement_Points:Measurement_Point_Round-SMD-Pad_Small" H 6150 2300 50  0001 C CNN
+F 3 "" H 6150 2300 50  0000 C CNN
+	1    6150 2300
+	0    1    1    0
+$EndComp
+$Comp
+L TEST TP6
+U 1 1 58E3853E
+P 2650 3200
+F 0 "TP6" H 2650 3500 50  0000 C BNN
+F 1 "TEST" H 2650 3450 50  0000 C CNN
+F 2 "Measurement_Points:Measurement_Point_Round-SMD-Pad_Small" H 2650 3200 50  0001 C CNN
+F 3 "" H 2650 3200 50  0000 C CNN
+	1    2650 3200
+	0    1    1    0
+$EndComp
+$Comp
+L TEST TP4
+U 1 1 58E38AD9
+P 2650 1800
+F 0 "TP4" H 2650 2100 50  0000 C BNN
+F 1 "TEST" H 2650 2050 50  0000 C CNN
+F 2 "Measurement_Points:Measurement_Point_Round-SMD-Pad_Small" H 2650 1800 50  0001 C CNN
+F 3 "" H 2650 1800 50  0000 C CNN
+	1    2650 1800
+	0    1    1    0
+$EndComp
 $EndSCHEMATC
