File: hardware/KiCAD/motors.sch (KiCad schematic (older format))
At the start: 49 parts, among them U10 AH3772, U11 AH3772, U12 AH3772, U5 MC33926PNB, U6 MC33926PNB, U7 Motor, U8 Motor, U9 AH3772

Commit message: Add LGA layouts for sensors
Parts:
- U5, U6: footprint (none) -> PiBot:PQFN-32-EP-0.8mm
Changed lines of the file:
@@
 F 0 "U5" H 4350 3300 60  0000 C CNN
 F 1 "MC33926PNB" V 3800 2300 60  0000 C CNB
-F 2 "" H 2650 3300 60  0001 C CNN
+F 2 "PiBot:PQFN-32-EP-0.8mm" H 2650 3300 60  0001 C CNN
 F 3 "" H 2650 3300 60  0001 C CNN
 	1    3800 2300
@@
 F 0 "U6" H 4350 6800 60  0000 C CNN
 F 1 "MC33926PNB" V 3800 5800 60  0000 C CNB
-F 2 "" H 2650 6800 60  0001 C CNN
+F 2 "PiBot:PQFN-32-EP-0.8mm" H 2650 6800 60  0001 C CNN
 F 3 "" H 2650 6800 60  0001 C CNN
 	1    3800 5800
