File: hardware/KiCAD/motors.sch (KiCad schematic (older format))
At the start: 37 parts

Commit message: Fix errors in schematic
- Fix motor feedback circuit
- Replace micro SD card with standard symbol
- Replace some 0ohm's with cuttable traces
- Clean up motor sheet
Parts:
- removed R? (x2): 0R, symbol R
- removed R?: 10k, symbol R
- added C? (x4): 1uF, symbol C
- added C? (x2): 10uF, symbol C
- added C? (x2): 0.1uF, symbol C
- added D? (x2): 3.3V, symbol D_Zener_Small
- added JP? (x2): Jumper_NC_Small, symbol Jumper_NC_Small
- added R? (x2): 100, symbol R
- added R?: 200, symbol R
- R?: value 10k -> 200
Connections:
- wire segments 166 -> 139
Other:
- note added: "Common Components"
- note added: "FB_L/R are feedback analog lines for\nsensing the amount of current the motor\ndriver is sending. The voltage measured \non this line divided by 0.48ohm will give\nthe motor current"
- note added: "Left Motor"
- note added: "Magnetic Motor Encoders"
- note added: "Right Motor"
- note removed: "FB_L/R are feedback analog lines for\nsensing the amount of current the motor\ndriver is sending. Solder the 0 ohm and\ndesolder the 10k to ground for use."
- moved on the sheet: C?

Commit message: Minor cleanup
Other:
- note added: "By:\nBroderick Carlin\nTyler Holmes"
- note added: "MIT License\n"
- note added: "PycoBot (Teensy uPython Robot)"
Changed lines of the file:
@@
 	9700 4200 9700 4100
 Connection ~ 9700 4100
+Text Notes 7050 7050 0    60   ~ 12
+By:\nBroderick Carlin\nTyler Holmes
+Text Notes 7950 7050 0    60   ~ 12
+MIT License\n
+Text Notes 7350 7500 0    60   ~ 12
+PycoBot (Teensy uPython Robot)
 $EndSCHEMATC

Commit message: Add MacroFab library and update SD card
Parts:
- C18, C19, C20, C21, C22, C23, C24, C25, C26, C27, C28, C29, C30, C31, C32, C33: renamed from C?; footprint (none) -> Capacitors_SMD:C_0402
- C34, C35: renamed from C?; footprint (none) -> Capacitors_SMD:C_1206
- R17, R18: renamed from R?; footprint (none) -> Resistors_SMD:R_0805
- R19, R20, R21, R22, R23, R24, R25, R26, R27: renamed from R?; footprint (none) -> Resistors_SMD:R_0402
- U10, U11, U12, U9: renamed from U?; footprint (none) -> TO_SOT_Packages_SMD:SOT-23
- gave numbers to parts that had none: 16

Commit message: adding in PQFN to motor controller
Parts:
- U5, U6: footprint (none) -> PiBot:PQFN-32-EP-0.8mm
Changed lines of the file:
@@
 LIBS:MF_Connectors
 LIBS:PiBot-cache
-EELAYER 25 0
+EELAYER 26 0
 EELAYER END
 $Descr A4 11693 8268
@@
 U 1 1 586EED1D
 P 7350 5900
-F 0 "C27" H 7375 6000 50  0000 L CNN
-F 1 "0.1uF" H 7375 5800 50  0000 L CNN
+F 0 "C27" H 7150 6000 50  0000 L CNN
+F 1 "0.1uF" H 7100 5800 50  0000 L CNN
 F 2 "Capacitors_SMD:C_0402" H 7388 5750 50  0001 C CNN
 F 3 "" H 7350 5900 50  0000 C CNN
@@
 U 1 1 586EED56
 P 9450 5900
-F 0 "C31" H 9475 6000 50  0000 L CNN
-F 1 "0.1uF" H 9475 5800 50  0000 L CNN
+F 0 "C31" H 9250 6000 50  0000 L CNN
+F 1 "0.1uF" H 9200 5800 50  0000 L CNN
 F 2 "Capacitors_SMD:C_0402" H 9488 5750 50  0001 C CNN
 F 3 "" H 9450 5900 50  0000 C CNN
@@
 U 1 1 586EED89
 P 7350 2600
-F 0 "C26" H 7375 2700 50  0000 L CNN
-F 1 "0.1uF" H 7375 2500 50  0000 L CNN
+F 0 "C26" H 7150 2700 50  0000 L CNN
+F 1 "0.1uF" H 7100 2500 50  0000 L CNN
 F 2 "Capacitors_SMD:C_0402" H 7388 2450 50  0001 C CNN
 F 3 "" H 7350 2600 50  0000 C CNN
@@
 U 1 1 586EEDB5
 P 9450 2600
-F 0 "C30" H 9475 2700 50  0000 L CNN
-F 1 "0.1uF" H 9475 2500 50  0000 L CNN
+F 0 "C30" H 9250 2700 50  0000 L CNN
+F 1 "0.1uF" H 9200 2500 50  0000 L CNN
 F 2 "Capacitors_SMD:C_0402" H 9488 2450 50  0001 C CNN
 F 3 "" H 9450 2600 50  0000 C CNN
@@
 F 0 "U5" H 4350 3300 60  0000 C CNN
 F 1 "MC33926PNB" V 3800 2300 60  0000 C CNB
-F 2 "" H 2650 3300 60  0001 C CNN
+F 2 "PiBot:PQFN-32-EP-0.8mm" H 2650 3300 60  0001 C CNN
 F 3 "" H 2650 3300 60  0001 C CNN
 	1    3800 2300
@@
 U 1 1 586F64D9
 P 2200 2650
-F 0 "C19" H 2100 2750 50  0000 L CNN
-F 1 "0.1uF" H 1950 2550 50  0000 L CNN
+F 0 "C19" V 2250 2700 50  0000 L CNN
+F 1 "0.1uF" V 2150 2700 50  0000 L CNN
 F 2 "Capacitors_SMD:C_0402" H 2238 2500 50  0001 C CNN
 F 3 "" H 2200 2650 50  0000 C CNN
@@
 F 0 "U6" H 4350 6800 60  0000 C CNN
 F 1 "MC33926PNB" V 3800 5800 60  0000 C CNB
-F 2 "" H 2650 6800 60  0001 C CNN
+F 2 "PiBot:PQFN-32-EP-0.8mm" H 2650 6800 60  0001 C CNN
 F 3 "" H 2650 6800 60  0001 C CNN
 	1    3800 5800
@@
 U 1 1 586FA847
 P 2150 6150
-F 0 "C18" H 2050 6250 50  0000 L CNN
-F 1 "0.1uF" H 1900 6050 50  0000 L CNN
+F 0 "C18" V 2200 6200 50  0000 L CNN
+F 1 "0.1uF" V 2100 6200 50  0000 L CNN
 F 2 "Capacitors_SMD:C_0402" H 2188 6000 50  0001 C CNN
 F 3 "" H 2150 6150 50  0000 C CNN
@@
 U 1 1 5872EE06
 P 4750 2300
-F 0 "C22" H 4650 2400 50  0000 L CNN
+F 0 "C22" H 4550 2400 50  0000 L CNN
 F 1 "0.1uF" H 4500 2200 50  0000 L CNN
 F 2 "Capacitors_SMD:C_0402" H 4788 2150 50  0001 C CNN
@@
 U 1 1 586D4AB9
 P 2200 3300
-F 0 "C20" H 2100 3400 50  0000 L CNN
-F 1 "1uF" H 1950 3200 50  0000 L CNN
+F 0 "C20" V 2150 3350 50  0000 L CNN
+F 1 "1uF" V 2250 3350 50  0000 L CNN
 F 2 "Capacitors_SMD:C_0402" H 2238 3150 50  0001 C CNN
 F 3 "" H 2200 3300 50  0000 C CNN
@@
 U 1 1 586D6275
 P 2200 6800
-F 0 "C21" H 2100 6900 50  0000 L CNN
-F 1 "1uF" H 1950 6700 50  0000 L CNN
+F 0 "C21" V 2150 6850 50  0000 L CNN
+F 1 "1uF" V 2250 6850 50  0000 L CNN
 F 2 "Capacitors_SMD:C_0402" H 2238 6650 50  0001 C CNN
 F 3 "" H 2200 6800 50  0000 C CNN

Commit message: Add battery footprint and assign feather footrprint
Changed lines of the file:
@@
 LIBS:MF_Connectors
 LIBS:PiBot-cache
-EELAYER 26 0
+EELAYER 25 0
 EELAYER END
 $Descr A4 11693 8268
@@
 U 1 1 586EED1D
 P 7350 5900
-F 0 "C27" H 7150 6000 50  0000 L CNN
-F 1 "0.1uF" H 7100 5800 50  0000 L CNN
+F 0 "C27" H 7375 6000 50  0000 L CNN
+F 1 "0.1uF" H 7375 5800 50  0000 L CNN
 F 2 "Capacitors_SMD:C_0402" H 7388 5750 50  0001 C CNN
 F 3 "" H 7350 5900 50  0000 C CNN
@@
 U 1 1 586EED56
 P 9450 5900
-F 0 "C31" H 9250 6000 50  0000 L CNN
-F 1 "0.1uF" H 9200 5800 50  0000 L CNN
+F 0 "C31" H 9475 6000 50  0000 L CNN
+F 1 "0.1uF" H 9475 5800 50  0000 L CNN
 F 2 "Capacitors_SMD:C_0402" H 9488 5750 50  0001 C CNN
 F 3 "" H 9450 5900 50  0000 C CNN
@@
 U 1 1 586EED89
 P 7350 2600
-F 0 "C26" H 7150 2700 50  0000 L CNN
-F 1 "0.1uF" H 7100 2500 50  0000 L CNN
+F 0 "C26" H 7375 2700 50  0000 L CNN
+F 1 "0.1uF" H 7375 2500 50  0000 L CNN
 F 2 "Capacitors_SMD:C_0402" H 7388 2450 50  0001 C CNN
 F 3 "" H 7350 2600 50  0000 C CNN
@@
 U 1 1 586EEDB5
 P 9450 2600
-F 0 "C30" H 9250 2700 50  0000 L CNN
-F 1 "0.1uF" H 9200 2500 50  0000 L CNN
+F 0 "C30" H 9475 2700 50  0000 L CNN
+F 1 "0.1uF" H 9475 2500 50  0000 L CNN
 F 2 "Capacitors_SMD:C_0402" H 9488 2450 50  0001 C CNN
 F 3 "" H 9450 2600 50  0000 C CNN
@@
 U 1 1 586F64D9
 P 2200 2650
-F 0 "C19" V 2250 2700 50  0000 L CNN
-F 1 "0.1uF" V 2150 2700 50  0000 L CNN
+F 0 "C19" H 2100 2750 50  0000 L CNN
+F 1 "0.1uF" H 1950 2550 50  0000 L CNN
 F 2 "Capacitors_SMD:C_0402" H 2238 2500 50  0001 C CNN
 F 3 "" H 2200 2650 50  0000 C CNN
@@
 U 1 1 586FA847
 P 2150 6150
-F 0 "C18" V 2200 6200 50  0000 L CNN
-F 1 "0.1uF" V 2100 6200 50  0000 L CNN
+F 0 "C18" H 2050 6250 50  0000 L CNN
+F 1 "0.1uF" H 1900 6050 50  0000 L CNN
 F 2 "Capacitors_SMD:C_0402" H 2188 6000 50  0001 C CNN
 F 3 "" H 2150 6150 50  0000 C CNN
@@
 U 1 1 5872EE06
 P 4750 2300
-F 0 "C22" H 4550 2400 50  0000 L CNN
+F 0 "C22" H 4650 2400 50  0000 L CNN
 F 1 "0.1uF" H 4500 2200 50  0000 L CNN
 F 2 "Capacitors_SMD:C_0402" H 4788 2150 50  0001 C CNN
@@
 U 1 1 586D4AB9
 P 2200 3300
-F 0 "C20" V 2150 3350 50  0000 L CNN
-F 1 "1uF" V 2250 3350 50  0000 L CNN
+F 0 "C20" H 2100 3400 50  0000 L CNN
+F 1 "1uF" H 1950 3200 50  0000 L CNN
 F 2 "Capacitors_SMD:C_0402" H 2238 3150 50  0001 C CNN
 F 3 "" H 2200 3300 50  0000 C CNN
@@
 U 1 1 586D6275
 P 2200 6800
-F 0 "C21" V 2150 6850 50  0000 L CNN
-F 1 "1uF" V 2250 6850 50  0000 L CNN
+F 0 "C21" H 2100 6900 50  0000 L CNN
+F 1 "1uF" H 1950 6700 50  0000 L CNN
 F 2 "Capacitors_SMD:C_0402" H 2238 6650 50  0001 C CNN
 F 3 "" H 2200 6800 50  0000 C CNN
