File: hardware/KiCAD/motors.sch (KiCad schematic (older format))
At the start: 49 parts, among them U10 AH3772, U11 AH3772, U12 AH3772, U5 MC33926PNB, U6 MC33926PNB, U7 Motor, U8 Motor, U9 AH3772

Commit message: Add the rest of the missing footprints, aside from motor
Parts:
- D11, D12: footprint (none) -> Diodes_SMD:SOD-323; Part Number (none) -> MM3Z3V3ST1G
- JP10, JP7, JP8, JP9: footprint (none) -> PiBot:Jumper-NO
- JP11, JP12, JP13, JP14, JP5, JP6: footprint (none) -> PiBot:Jumper-NC
Changed lines of the file:
@@
 $EndComp
 $Comp
-L GND #PWR065
+L GND #PWR043
 U 1 1 586ED635
 P 6050 6000
-F 0 "#PWR065" H 6050 5750 50  0001 C CNN
+F 0 "#PWR043" H 6050 5750 50  0001 C CNN
 F 1 "GND" H 6050 5850 50  0001 C CNN
 F 2 "" H 6050 6000 50  0000 C CNN
@@
 $EndComp
 $Comp
-L GND #PWR066
+L GND #PWR044
 U 1 1 586ED63B
 P 6050 2500
-F 0 "#PWR066" H 6050 2250 50  0001 C CNN
+F 0 "#PWR044" H 6050 2250 50  0001 C CNN
 F 1 "GND" H 6050 2350 50  0001 C CNN
 F 2 "" H 6050 2500 50  0000 C CNN
@@
 F 0 "JP7" H 5900 2080 50  0000 C CNN
 F 1 "Jumper_NO_Small" H 5910 1940 50  0001 C CNN
-F 2 "" H 5900 2000 50  0001 C CNN
+F 2 "PiBot:Jumper-NO" H 5900 2000 50  0001 C CNN
 F 3 "" H 5900 2000 50  0000 C CNN
 	1    5900 2000
@@
 F 0 "JP8" H 5900 2680 50  0000 C CNN
 F 1 "Jumper_NO_Small" H 5910 2540 50  0001 C CNN
-F 2 "" H 5900 2600 50  0001 C CNN
+F 2 "PiBot:Jumper-NO" H 5900 2600 50  0001 C CNN
 F 3 "" H 5900 2600 50  0000 C CNN
 	1    5900 2600
@@
 F 0 "JP9" H 5900 5580 50  0000 C CNN
 F 1 "Jumper_NO_Small" H 5910 5440 50  0001 C CNN
-F 2 "" H 5900 5500 50  0001 C CNN
+F 2 "PiBot:Jumper-NO" H 5900 5500 50  0001 C CNN
 F 3 "" H 5900 5500 50  0000 C CNN
 	1    5900 5500
@@
 F 0 "JP10" H 5900 6180 50  0000 C CNN
 F 1 "Jumper_NO_Small" H 5910 6040 50  0001 C CNN
-F 2 "" H 5900 6100 50  0001 C CNN
+F 2 "PiBot:Jumper-NO" H 5900 6100 50  0001 C CNN
 F 3 "" H 5900 6100 50  0000 C CNN
 	1    5900 6100
@@
 F 0 "JP12" H 8250 5680 50  0000 C CNN
 F 1 "Jumper_NC_Small" H 8260 5540 50  0001 C CNN
-F 2 "" H 8250 5600 50  0001 C CNN
+F 2 "PiBot:Jumper-NC" H 8250 5600 50  0001 C CNN
 F 3 "" H 8250 5600 50  0000 C CNN
 	1    8250 5600
@@
 $EndComp
 $Comp
-L GND #PWR067
+L GND #PWR045
 U 1 1 586EED32
 P 7750 6150
-F 0 "#PWR067" H 7750 5900 50  0001 C CNN
+F 0 "#PWR045" H 7750 5900 50  0001 C CNN
 F 1 "GND" H 7750 6000 50  0001 C CNN
 F 2 "" H 7750 6150 50  0000 C CNN
@@
 F 0 "JP14" H 10350 5680 50  0000 C CNN
 F 1 "Jumper_NC_Small" H 10360 5540 50  0001 C CNN
-F 2 "" H 10350 5600 50  0001 C CNN
+F 2 "PiBot:Jumper-NC" H 10350 5600 50  0001 C CNN
 F 3 "" H 10350 5600 50  0000 C CNN
 	1    10350 5600
@@
 $EndComp
 $Comp
-L GND #PWR068
+L GND #PWR046
 U 1 1 586EED6B
 P 9850 6150
-F 0 "#PWR068" H 9850 5900 50  0001 C CNN
+F 0 "#PWR046" H 9850 5900 50  0001 C CNN
 F 1 "GND" H 9850 6000 50  0001 C CNN
 F 2 "" H 9850 6150 50  0000 C CNN
@@
 F 0 "JP11" H 8250 2380 50  0000 C CNN
 F 1 "Jumper_NC_Small" H 8260 2240 50  0001 C CNN
-F 2 "" H 8250 2300 50  0001 C CNN
+F 2 "PiBot:Jumper-NC" H 8250 2300 50  0001 C CNN
 F 3 "" H 8250 2300 50  0000 C CNN
 	1    8250 2300
@@
 $EndComp
 $Comp
-L GND #PWR069
+L GND #PWR047
 U 1 1 586EED9E
 P 7750 2850
-F 0 "#PWR069" H 7750 2600 50  0001 C CNN
+F 0 "#PWR047" H 7750 2600 50  0001 C CNN
 F 1 "GND" H 7750 2700 50  0001 C CNN
 F 2 "" H 7750 2850 50  0000 C CNN
@@
 F 0 "JP13" H 10350 2380 50  0000 C CNN
 F 1 "Jumper_NC_Small" H 10360 2240 50  0001 C CNN
-F 2 "" H 10350 2300 50  0001 C CNN
+F 2 "PiBot:Jumper-NC" H 10350 2300 50  0001 C CNN
 F 3 "" H 10350 2300 50  0000 C CNN
 	1    10350 2300
@@
 $EndComp
 $Comp
-L GND #PWR070
+L GND #PWR048
 U 1 1 586EEDCA
 P 9850 2850
-F 0 "#PWR070" H 9850 2600 50  0001 C CNN
+F 0 "#PWR048" H 9850 2600 50  0001 C CNN
 F 1 "GND" H 9850 2700 50  0001 C CNN
 F 2 "" H 9850 2850 50  0000 C CNN
@@
 $EndComp
 $Comp
-L GND #PWR071
+L GND #PWR049
 U 1 1 586F5981
 P 2500 2350
-F 0 "#PWR071" H 2500 2100 50  0001 C CNN
+F 0 "#PWR049" H 2500 2100 50  0001 C CNN
 F 1 "GND" H 2500 2200 50  0001 C CNN
 F 2 "" H 2500 2350 50  0000 C CNN
@@
 	2850 3150 2950 3150
 $Comp
-L GND #PWR072
+L GND #PWR050
 U 1 1 586F6FCF
 P 3150 3600
-F 0 "#PWR072" H 3150 3350 50  0001 C CNN
+F 0 "#PWR050" H 3150 3350 50  0001 C CNN
 F 1 "GND" H 3150 3450 50  0001 C CNN
 F 2 "" H 3150 3600 50  0000 C CNN
@@
 Connection ~ 3150 3500
 $Comp
-L GNDPWR #PWR073
+L GNDPWR #PWR051
 U 1 1 586F7492
 P 3950 3600
-F 0 "#PWR073" H 3950 3400 50  0001 C CNN
+F 0 "#PWR051" H 3950 3400 50  0001 C CNN
 F 1 "GNDPWR" H 3950 3470 50  0000 C CNN
 F 2 "" H 3950 3550 50  0000 C CNN
@@
 $EndComp
 $Comp
-L GND #PWR074
+L GND #PWR052
 U 1 1 586FA83E
 P 2500 5850
-F 0 "#PWR074" H 2500 5600 50  0001 C CNN
+F 0 "#PWR052" H 2500 5600 50  0001 C CNN
 F 1 "GND" H 2500 5700 50  0001 C CNN
 F 2 "" H 2500 5850 50  0000 C CNN
@@
 	2850 6650 2950 6650
 $Comp
-L GND #PWR075
+L GND #PWR053
 U 1 1 586FA871
 P 3150 7100
-F 0 "#PWR075" H 3150 6850 50  0001 C CNN
+F 0 "#PWR053" H 3150 6850 50  0001 C CNN
 F 1 "GND" H 3150 6950 50  0001 C CNN
 F 2 "" H 3150 7100 50  0000 C CNN
@@
 Connection ~ 3150 7000
 $Comp
-L GNDPWR #PWR076
+L GNDPWR #PWR054
 U 1 1 586FA87D
 P 3950 7100
-F 0 "#PWR076" H 3950 6900 50  0001 C CNN
+F 0 "#PWR054" H 3950 6900 50  0001 C CNN
 F 1 "GNDPWR" H 3950 6970 50  0000 C CNN
 F 2 "" H 3950 7050 50  0000 C CNN
@@
 F 0 "D11" H 1900 3390 50  0000 C CNN
 F 1 "3.3V" H 1900 3210 50  0000 C CNN
-F 2 "" V 1900 3300 50  0001 C CNN
+F 2 "Diodes_SMD:SOD-323" V 1900 3300 50  0001 C CNN
 F 3 "" V 1900 3300 50  0000 C CNN
+F 4 "MM3Z3V3ST1G" H 1900 3300 60  0001 C CNN "Part Number"
 	1    1900 3300
 	0    1    1    0
@@
 F 0 "D12" H 1900 6890 50  0000 C CNN
 F 1 "3.3V" H 1900 6710 50  0000 C CNN
-F 2 "" V 1900 6800 50  0001 C CNN
+F 2 "Diodes_SMD:SOD-323" V 1900 6800 50  0001 C CNN
 F 3 "" V 1900 6800 50  0000 C CNN
+F 4 "MM3Z3V3ST1G" H 1900 6800 60  0001 C CNN "Part Number"
 	1    1900 6800
 	0    1    1    0
@@
 F 0 "JP5" H 1700 3030 50  0000 C CNN
 F 1 "Jumper_NC_Small" H 1710 2890 50  0001 C CNN
-F 2 "" H 1700 2950 50  0001 C CNN
+F 2 "PiBot:Jumper-NC" H 1700 2950 50  0001 C CNN
 F 3 "" H 1700 2950 50  0000 C CNN
 	1    1700 2950
@@
 F 0 "JP6" H 1700 6530 50  0000 C CNN
 F 1 "Jumper_NC_Small" H 1710 6390 50  0001 C CNN
-F 2 "" H 1700 6450 50  0001 C CNN
+F 2 "PiBot:Jumper-NC" H 1700 6450 50  0001 C CNN
 F 3 "" H 1700 6450 50  0000 C CNN
 	1    1700 6450
@@
 +VBatt
 $Comp
-L GNDPWR #PWR077
+L GNDPWR #PWR055
 U 1 1 586EDCC3
 P 9700 4200
-F 0 "#PWR077" H 9700 4000 50  0001 C CNN
+F 0 "#PWR055" H 9700 4000 50  0001 C CNN
 F 1 "GNDPWR" H 9700 4070 50  0000 C CNN
 F 2 "" H 9700 4150 50  0000 C CNN

Commit message: Dry positioning of large portion of the components
Parts:
- U7, U8: footprint (none) -> PiBot:Sanyo_GearMotor
Changed lines of the file:
@@
 F 0 "U7" H 5550 2550 60  0000 C CNN
 F 1 "Motor" V 5300 2300 60  0000 C CNB
-F 2 "" H 4900 1750 60  0001 C CNN
+F 2 "PiBot:Sanyo_GearMotor" H 4900 1750 60  0001 C CNN
 F 3 "" H 4900 1750 60  0001 C CNN
 	1    5350 2300
@@
 F 0 "U8" H 5550 6050 60  0000 C CNN
 F 1 "Motor" V 5300 5800 60  0000 C CNB
-F 2 "" H 4900 5250 60  0001 C CNN
+F 2 "PiBot:Sanyo_GearMotor" H 4900 5250 60  0001 C CNN
 F 3 "" H 4900 5250 60  0001 C CNN
 	1    5350 5800
