File: hardware/KiCAD/PiBot.kicad_pcb (KiCad board)
At the start: 2 copper layers, 64 x 123 mm, 177 parts, among them P2 CONN_02X05, P3 I2C_EXPANSION, P5 Feather-Adaper, SW1 SPST, SW2 SW_SPDT, SW3 SW_SPDT, SW4 SW_SPDT, SW5 SW_SPDT, U1 DMG2302U, U10 AH3772, U11 AH3772, U12 AH3772, U13 BH1745NUC, U14 BH1745NUC, U15 L3GD20H, U16 LSM303DLHCTR, U17 N-FET, U2 MKL03ZxxVFK4, U3 N-FET, U4 TPS63060, U5 MC33926PNB, U6 MC33926PNB, U7 Motor, U8 Motor, U9 AH3772

Commit message: More routing
Parts:
- R4, R5: moved to F.Cu
- moved TP35 165.3 mm to (158.0, 26.5)
- moved TP41 155.3 mm to (153.0, 26.0)
- moved TP49 153.0 mm to (147.0, 25.5)
- moved TP10 90.2 mm to (125.2, 82.5)
- moved TP12 81.1 mm to (125.2, 85.5)
- moved TP47 76.8 mm to (128.5, 25.5)
- moved TP14 73.1 mm to (100.0, 143.0)
- moved P3 51.3 mm to (125.5, 106.5), turned to 90 degrees
- moved C37 44.0 mm to (158.0, 146.8)
- moved C41 36.4 mm to (156.0, 93.0)
- moved U15 36.3 mm to (155.0, 90.0)
- moved C42 34.5 mm to (151.8, 92.5)
- moved C43 34.4 mm to (150.0, 92.5)
- moved C40 34.0 mm to (147.8, 92.8)
- moved R24 30.4 mm to (166.6, 137.6), turned to 0 degrees
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Routing:
- net SCL: track 0.00 -> 166.4 mm, vias 0 -> 7
- net SDA: track 0.00 -> 162.4 mm, vias 0 -> 7
- net Net-(R28-Pad1): track 0.00 -> 71.5 mm, vias 0 -> 2
- net Net-(TP10-Pad1): track 0.00 -> 33.2 mm, vias 0 -> 1
- net Net-(TP12-Pad1): track 0.00 -> 30.9 mm, vias 0 -> 1
- net Net-(JP15-Pad1): track 0.00 -> 30.0 mm, vias 0 -> 1
- net rear_bumper: track 0.00 -> 11.9 mm
- net front_bumper: track 0.00 -> 5.26 mm
- net Net-(TP4-Pad1): track 0.00 -> 5.26 mm, vias 0 -> 1
- net Net-(TP6-Pad1): track 0.00 -> 3.57 mm, vias 0 -> 1
- net +3V3: track 56.6 -> 59.2 mm, vias 2 -> 4
- net Net-(C41-Pad1): track 0.00 -> 1.80 mm
- net /I2C_LSB_BIT: track 7.21 -> 8.64 mm
- net Net-(DRDY1-Pad1): track 17.3 -> 18.4 mm
Other:
- net class Default: trace_width 0.4 -> 0.25
